File: avionics/flight computer FOX/flight computer FOX.kicad_sch (KiCad schematic)
At the start: 5 parts, among them U1 ESP32-S3-DevKitC

Commit message: kicad
Parts:
- added A1: BMP280_Module, Charleslabs_Parts:BMP280_Module, symbol Charleslabs_Parts:BMP280_Module
- added A2: MPU6050_Module, Charleslabs_Parts:MPU6050_Module, symbol Charleslabs_Parts:MPU6050_Module
Changed lines of the file:
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@@
+    )
+  )
+  (symbol (lib_id "Charleslabs_Parts:MPU6050_Module") (at 63.5 58.42 0) (unit 1)
+    (in_bom yes) (on_board yes) (dnp no) (fields_autoplaced)
+    (property "Reference" "A2" (at 80.01 54.5339 0)
+      (effects (font (size 1.27 1.27)))
+    )
+    (property "Value" "MPU6050_Module" (at 80.01 57.0739 0)
+      (effects (font (size 1.27 1.27)))
+    )
+    (property "Footprint" "Charleslabs_Parts:MPU6050_Module" (at 87.63 48.26 0)
+      (effects (font (size 1.27 1.27)) hide)
+    )
+    (property "Datasheet" "" (at 57.15 46.99 0)
+      (effects (font (size 1.27 1.27)) hide)
+    )
+    (pin "1")
+    (pin "2")
+    (pin "3")
+    (pin "4")
+    (pin "5")
+    (pin "6")
+    (pin "7")
+    (pin "8")
+    (instances
+      (project "flight computer FOX"
+        (path "/05785e23-8de8-49cd-8fd9-ec33b4a12221"
+          (reference "A2") (unit 1)
+        )
+      )
     )
   )
@@
         )
       )
+    )
+  )
+  (symbol (lib_id "Charleslabs_Parts:BMP280_Module") (at 62.23 115.57 0) (unit 1)
+    (in_bom yes) (on_board yes) (dnp no) (fields_autoplaced)
+    (property "Reference" "A1" (at 68.58 114.3 0)
+      (effects (font (size 1.27 1.27)) (justify left))
+    )
+    (property "Value" "BMP280_Module" (at 68.58 116.84 0)
+      (effects (font (size 1.27 1.27)) (justify left))
+    )
+    (property "Footprint" "Charleslabs_Parts:BMP280_Module" (at 83.82 109.22 0)
+      (effects (font (size 1.27 1.27)) hide)
+    )
+    (property "Datasheet" "" (at 57.15 104.14 0)
+      (effects (font (size 1.27 1.27)) hide)
+    )
+    (pin "1")
+    (pin "2")
+    (pin "3")
+    (pin "4")
+    (pin "5")
+    (pin "6")
+    (instances
+      (project "flight computer FOX"
+        (path "/05785e23-8de8-49cd-8fd9-ec33b4a12221"
+          (reference "A1") (unit 1)
+        )
+      )

Commit message: some stuff
Parts:
- added C5, C6: 0.01uf, symbol Device:C
- added U2: LM7805_TO220, Package_TO_SOT_THT:TO-220-3_Vertical, symbol Regulator_Linear:LM7805_TO220
Connections:
- net +5V: now also A1.1 (VCC), A2.1 (VCC), C5.1, C6.1, U2.3 (VO)
- net GND: now also A1.2 (GND), A2.2 (GND), C5.2, C6.2, U2.2 (GND)
- net SCL: now reaches A2.3 (SCL)
- net SCL: now also A1.3 (SCL)
- net SDA: now reaches A2.4 (SDA)
- net SDA: now also A1.4 (SDA)
- net XDA: now reaches A2.5 (XDA)
- net XDA: now also A1.5 (CSB)
- net XCL: now reaches A2.6 (XCL)
- net XCL: now also A1.6 (SD0)
- new net +BATT: U2.1 (VI)
Other:
- moved on the sheet: C1, C2, C3, C4, U1

Commit message: more flight computer work
Parts:
- added BZ1: Buzzer, Buzzer_Beeper:Buzzer_12x9.5RM7.6, symbol Device:Buzzer
- added C7: 0.33uf, Capacitor_SMD:C_0805_2012Metric_Pad1.18x1.45mm_HandSolder, symbol Device:C
- added C8: 0.1uf, Capacitor_SMD:C_0805_2012Metric_Pad1.18x1.45mm_HandSolder, symbol Device:C
- added D1: LED_BGRK, LED_THT:LED_D5.0mm-4_RGB, symbol Device:LED_BGRK
- added R1: R1k, symbol Device:R
- added R2, R3: R10k, symbol Device:R
- C1, C2, C3, C4, C5, C6: footprint (none) -> Capacitor_SMD:C_0805_2012Metric_Pad1.18x1.45mm_HandSolder
Connections:
- net +5V: now also C8.2, R2.2, R3.2
- net +BATT: now also C7.2
- net GND: now also BZ1.2 (+), C7.1, C8.1, R1.1
- net SCL: now also R2.1
- net SDA: now also R3.1
- new net: D1.4 (K), R1.2
- new net blueled: D1.1 (BA)
- new net buzzer: BZ1.1 (-)
- new net greenled: D1.2 (GA)
- new net redled: D1.3 (RA)
Other:
- moved on the sheet: C1, C2, C3, C4, U1

Commit message: more avionics work
Parts:
- removed U1: ESP32-S3-DevKitC, Espressif:ESP32-S3-DevKitC, symbol Espressif:ESP32-S3-DevKitC
- added C9: 1uf, Capacitor_SMD:C_0805_2012Metric_Pad1.18x1.45mm_HandSolder, symbol Device:C
- added J1: Screw_Terminal_01x02, TerminalBlock:TerminalBlock_bornier-2_P5.08mm, symbol Connector:Screw_Terminal_01x02
- added U1: ESP32-DevKitC, Espressif:ESP32-DevKitC, symbol Espressif:ESP32-DevKitC
- added U3: NRF24L01_Breakout, RF_Module:nRF24L01_Breakout, symbol RF:NRF24L01_Breakout
- C1, C2, C3, C4, C5, C6: value 0.01uf -> 1uf
- R1, R2, R3: footprint (none) -> Resistor_SMD:R_0805_2012Metric_Pad1.20x1.40mm_HandSolder
Connections:
- net +3V3: now also U1.1 (3V3)
- net +5V: now also C9.1, U1.19 (5V), U3.2 (VCC)
- net +BATT: now also J1.1 (Pin_1)
- net GND: now also A2.7 (AD0), C9.2, J1.2 (Pin_2), U1.14 (GND), U1.32 (GND), U1.38 (GND), U3.1 (GND)
- net SCL: now also U1.36 (GPIO22)
- net SDA: now also U1.33 (GPIO21)
- net blueled: now also U1.23 (*MTDO/GPIO15/ADC2_CH3)
- net buzzer: now also U1.8 (32K_XN/GPIO33/ADC1_CH5)
- net greenled: now also U1.12 (MTMS/GPIO14/ADC2_CH6)
- net redled: now also U1.15 (MTCK/GPIO13/ADC2_CH4)
- net INTMPU: now reaches A2.8 (INT)
- net INTMPU: now also U1.9 (DAC_1/ADC2_CH8/GPIO25)
- net XCL: no longer names the net of A2.6 (XCL)
- net XCL: no longer A1.6 (SD0)
- net XDA: no longer names the net of A2.5 (XDA)
- net XDA: no longer A1.5 (CSB)
- new net CE: U1.11 (ADC2_CH7/GPIO27), U3.3 (CE)
- new net CS: U1.29 (*GPIO5), U3.4 (~{CSN})
- new net INTNRF: U1.10 (DAC_2/ADC2_CH9/GPIO26), U3.8 (IRQ)
- new net MISO: U1.31 (GPIO19), U3.7 (MISO)
- new net MOSI: U1.37 (GPIO23), U3.6 (MOSI)
- new net SCK: U1.30 (GPIO18), U3.5 (SCK)
Other:
- moved on the sheet: C1, C2, C3, C4, C7, C8, U2

Commit message: hmm
Changed lines of the file:
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@@
     (stroke (width 0) (type default))
   )
-  (wire (pts (xy 149.86 138.43) (xy 146.05 138.43))
+  (wire (pts (xy 152.4 138.43) (xy 146.05 138.43))
     (stroke (width 0) (type default))
   )
@@
     )
   )
-  (symbol (lib_id "power:+5V") (at 149.86 138.43 270) (unit 1)
-    (in_bom yes) (on_board yes) (dnp no) (fields_autoplaced)
-    (property "Reference" "#PWR012" (at 146.05 138.43 0)
-      (effects (font (size 1.27 1.27)) hide)
-    )
-    (property "Value" "+5V" (at 153.67 138.43 90)
+  (symbol (lib_id "power:+5V") (at 152.4 138.43 270) (unit 1)
+    (in_bom yes) (on_board yes) (dnp no) (fields_autoplaced)
+    (property "Reference" "#PWR012" (at 148.59 138.43 0)
+      (effects (font (size 1.27 1.27)) hide)
+    )
+    (property "Value" "+5V" (at 156.21 138.43 90)
       (effects (font (size 1.27 1.27)) (justify left))
     )
-    (property "Footprint" "" (at 149.86 138.43 0)
-      (effects (font (size 1.27 1.27)) hide)
-    )
-    (property "Datasheet" "" (at 149.86 138.43 0)
-      (effects (font (size 1.27 1.27)) hide)
-    )
+    (property "Footprint" "" (at 152.4 138.43 0)
+      (effects (font (size 1.27 1.27)) hide)
+    )
+    (property "Datasheet" "" (at 152.4 138.43 0)
+      (effects (font (size 1.27 1.27)) hide)
+    )

Commit message: more kicad
Parts:
- removed R2, R3: R10k, Resistor_SMD:R_0805_2012Metric_Pad1.20x1.40mm_HandSolder, symbol Device:R
Changed lines of the file:
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@@
-    )
-  )
-  (global_label "SDA" (shape input) (at 127 46.99 270) (fields_autoplaced)
-    (effects (font (size 1.27 1.27)) (justify right))
-    (property "Intersheetrefs" "${INTERSHEET_REFS}" (at 127 53.4639 90)
-      (effects (font (size 1.27 1.27)) (justify right) hide)
     )
   )
@@
     (effects (font (size 1.27 1.27)) (justify right))
     (property "Intersheetrefs" "${INTERSHEET_REFS}" (at 48.1966 53.34 0)
-      (effects (font (size 1.27 1.27)) (justify right) hide)
-    )
-  )
-  (global_label "SCL" (shape input) (at 118.11 46.99 270) (fields_autoplaced)
-    (effects (font (size 1.27 1.27)) (justify right))
-    (property "Intersheetrefs" "${INTERSHEET_REFS}" (at 118.11 53.4034 90)
       (effects (font (size 1.27 1.27)) (justify right) hide)
     )
@@
     )
   )
-  (symbol (lib_id "Device:R") (at 118.11 43.18 180) (unit 1)
-    (in_bom yes) (on_board yes) (dnp no) (fields_autoplaced)
-    (property "Reference" "R2" (at 120.65 42.545 0)
-      (effects (font (size 1.27 1.27)) (justify right))
-    )
-    (property "Value" "R10k" (at 120.65 45.085 0)
-      (effects (font (size 1.27 1.27)) (justify right))
-    )
-    (property "Footprint" "Resistor_SMD:R_0805_2012Metric_Pad1.20x1.40mm_HandSolder" (at 119.888 43.18 90)
-      (effects (font (size 1.27 1.27)) hide)
-    )
-    (property "Datasheet" "~" (at 118.11 43.18 0)
-      (effects (font (size 1.27 1.27)) hide)
-    )
-    (pin "1")
-    (pin "2")
-    (instances
-      (project "flight computer FOX"
-        (path "/05785e23-8de8-49cd-8fd9-ec33b4a12221"
-          (reference "R2") (unit 1)
-        )
-      )
-    )
-  )
-  (symbol (lib_id "power:+5V") (at 127 39.37 0) (unit 1)
-    (in_bom yes) (on_board yes) (dnp no) (fields_autoplaced)
-    (property "Reference" "#PWR018" (at 127 43.18 0)
-      (effects (font (size 1.27 1.27)) hide)
-    )
-    (property "Value" "+5V" (at 127 34.29 0)
-      (effects (font (size 1.27 1.27)))
-    )
-    (property "Footprint" "" (at 127 39.37 0)
-      (effects (font (size 1.27 1.27)) hide)
-    )
-    (property "Datasheet" "" (at 127 39.37 0)
-      (effects (font (size 1.27 1.27)) hide)
-    )
-    (pin "1")
-    (instances
-      (project "flight computer FOX"
-        (path "/05785e23-8de8-49cd-8fd9-ec33b4a12221"
-          (reference "#PWR018") (unit 1)
-        )
-      )
-    )
-  )
   (symbol (lib_id "power:GND") (at 62.23 128.27 0) (unit 1)
     (in_bom yes) (on_board yes) (dnp no) (fields_autoplaced)
@@
     )
   )
-  (symbol (lib_id "power:+5V") (at 118.11 39.37 0) (unit 1)
-    (in_bom yes) (on_board yes) (dnp no) (fields_autoplaced)
-    (property "Reference" "#PWR017" (at 118.11 43.18 0)
-      (effects (font (size 1.27 1.27)) hide)
-    )
-    (property "Value" "+5V" (at 118.11 34.29 0)
-      (effects (font (size 1.27 1.27)))
-    )
-    (property "Footprint" "" (at 118.11 39.37 0)
-      (effects (font (size 1.27 1.27)) hide)
-    )
-    (property "Datasheet" "" (at 118.11 39.37 0)
-      (effects (font (size 1.27 1.27)) hide)
-    )
-    (pin "1")
-    (instances
-      (project "flight computer FOX"
-        (path "/05785e23-8de8-49cd-8fd9-ec33b4a12221"
-          (reference "#PWR017") (unit 1)
-        )
-      )
-    )
-  )
   (symbol (lib_id "Device:C") (at 203.2 48.26 90) (unit 1)
     (in_bom yes) (on_board yes) (dnp no)
@@
         )
       )
-    )
-  )
-  (symbol (lib_id "Device:R") (at 127 43.18 180) (unit 1)
-    (in_bom yes) (on_board yes) (dnp no) (fields_autoplaced)
-    (property "Reference" "R3" (at 129.54 42.545 0)
-      (effects (font (size 1.27 1.27)) (justify right))
-    )
-    (property "Value" "R10k" (at 129.54 45.085 0)
-      (effects (font (size 1.27 1.27)) (justify right))
-    )
-    (property "Footprint" "Resistor_SMD:R_0805_2012Metric_Pad1.20x1.40mm_HandSolder" (at 128.778 43.18 90)
-      (effects (font (size 1.27 1.27)) hide)
-    )
-    (property "Datasheet" "~" (at 127 43.18 0)
-      (effects (font (size 1.27 1.27)) hide)
-    )
-    (pin "1")
-    (pin "2")
-    (instances
-      (project "flight computer FOX"
-        (path "/05785e23-8de8-49cd-8fd9-ec33b4a12221"
-          (reference "R3") (unit 1)
-        )
-      )

Commit message: fox v1
Parts:
- removed BZ1: Buzzer, Buzzer_Beeper:Buzzer_12x9.5RM7.6, symbol Device:Buzzer
- added J2, J3, J4, J5, J6: Conn_01x03, Connector_PinHeader_2.54mm:PinHeader_1x03_P2.54mm_Vertical, symbol Connector_Generic:Conn_01x03
- D1: footprint LED_THT:LED_D5.0mm-4_RGB -> LED_THT:LED_D5.0mm-4_RGB_Wide_Pins
Connections:
- net buzzer is gone; now on net redled: U1.8 (32K_XN/GPIO33/ADC1_CH5)
- net +5V: now also J2.2 (Pin_2), J3.2 (Pin_2), J4.2 (Pin_2), J5.2 (Pin_2)
- net GND: now also J2.3 (Pin_3), J3.3 (Pin_3), J4.3 (Pin_3), J5.3 (Pin_3), J6.3 (Pin_3)
- net INTMPU: now also U1.5 (VDET_1/GPIO34/ADC1_CH6); no longer U1.9 (DAC_1/ADC2_CH8/GPIO25)
- net INTNRF: now also U1.6 (VDET_2/GPIO35/ADC1_CH7); no longer U1.10 (DAC_2/ADC2_CH9/GPIO26)
- net SCL: now also J6.2 (Pin_2)
- net SDA: now also J6.1 (Pin_1)
- net greenled: now also U1.7 (32K_XP/GPIO32/ADC1_CH4); no longer U1.12 (MTMS/GPIO14/ADC2_CH6)
- net redled: no longer U1.15 (MTCK/GPIO13/ADC2_CH4)
- new net servoout1: J2.1 (Pin_1), U1.9 (DAC_1/ADC2_CH8/GPIO25)
- new net servoout2: J3.1 (Pin_1), U1.10 (DAC_2/ADC2_CH9/GPIO26)
- new net servoout3: J4.1 (Pin_1), U1.12 (MTMS/GPIO14/ADC2_CH6)
- new net servoout4: J5.1 (Pin_1), U1.15 (MTCK/GPIO13/ADC2_CH4)

Commit message: FLIGHT Compupdate
Parts:
- removed C9: 1uf, Capacitor_SMD:C_0805_2012Metric_Pad1.18x1.45mm_HandSolder, symbol Device:C
- removed U3: NRF24L01_Breakout, RF_Module:nRF24L01_Breakout, symbol RF:NRF24L01_Breakout
- added BZ1: Buzzer, Buzzer_Beeper:Buzzer_12x9.5RM7.6, symbol Device:Buzzer
Connections:
- net +3V3: now also A1.1 (VCC), A2.1 (VCC), C5.1, C6.1
- net +5V: no longer A1.1 (VCC), A2.1 (VCC), C5.1, C6.1
- net GND: now also BZ1.2 (+)
- net CE: no longer names the net of U1.11 (ADC2_CH7/GPIO27)
- net CS: no longer names the net of U1.29 (*GPIO5)
- net INTNRF renamed buzzer
- net buzzer: now also BZ1.1 (-)
- net MISO: no longer names the net of U1.31 (GPIO19)
- net SCK: no longer names the net of U1.30 (GPIO18)
