File: avionics/flight computer FOX/flight computer FOX.kicad_pcb (KiCad board)
At the start: 4 copper layers, 45.1 x 68.6 mm, 20 parts, among them J1 Screw_Terminal_01x02, U1 ESP32-DevKitC, U2 LM7805_TO220, U3 NRF24L01_Breakout

Commit message: hmm
Routing:
- net SDA: track 0.00 -> 5.08 mm
Changed lines of the file:
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@@
   (segment (start 59.9225 27.94) (end 62.4625 30.48) (width 1) (layer "B.Cu") (net 5))
   (segment (start 65.04 50.8) (end 62.87 50.8) (width 1) (layer "B.Cu") (net 9))
+  (segment (start 59.69 63.5) (end 64.77 63.5) (width 0.25) (layer "B.Cu") (net 31))
   (segment (start 32.81 73.66) (end 32.72 73.75) (width 0.25) (layer "B.Cu") (net 42))
   (zone (net 4) (net_name "+5V") (layer "In1.Cu") (hatch edge 0.5)

Commit message: more kicad
Parts:
- removed R2, R3: R10k, Resistor_SMD:R_0805_2012Metric_Pad1.20x1.40mm_HandSolder
- U2: moved to F.Cu
- moved C6 59.8 mm to (32.4, 86.4)
- moved BZ1 57.0 mm to (47.6, 26.0)
- moved C9 40.0 mm to (43.2, 31.8), turned to 180 degrees
- moved J1 36.2 mm to (31.8, 28.6)
- moved A2 34.3 mm to (60.3, 21.6)
- moved U3 31.4 mm to (59.8, 81.6), turned to 90 degrees
- moved C2 30.2 mm to (59.7, 48.9)
- moved C7 26.7 mm to (36.8, 31.8)
- moved R1 23.4 mm to (50.2, 33.7), turned to 0 degrees
- moved C5 20.7 mm to (58.8, 76.2), turned to 180 degrees
- moved U2 20.0 mm to (39.7, 27.9)
- moved U1 20.0 mm to (28.6, 41.3)
- moved A1 18.6 mm to (58.4, 51.6), turned to 90 degrees
- moved C8 18.5 mm to (45.1, 21.0)
- moved D1 17.1 mm to (54.6, 34.3), turned to -90 degrees
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Connections:
- U1 pad 12: unconnected-(U1-MTMS/GPIO14/ADC2_CH6-Pad12) -> greenled
- U1 pad 15: unconnected-(U1-MTCK/GPIO13/ADC2_CH4-Pad15) -> redled
- U1 pad 23: unconnected-(U1-*MTDO/GPIO15/ADC2_CH3-Pad23) -> blueled
Routing:
- net MOSI: track 0.00 -> 60.8 mm
- net redled: track 0.00 -> 56.4 mm, vias 0 -> 3
- net greenled: track 0.00 -> 54.0 mm, vias 0 -> 1
- net blueled: track 0.00 -> 53.2 mm, vias 0 -> 2
- net CE: track 0.00 -> 47.2 mm
- net INTNRF: track 0.00 -> 46.4 mm
- net INTMPU: track 0.00 -> 41.0 mm
- net buzzer: track 0.00 -> 40.9 mm
- net MISO: track 0.00 -> 40.2 mm
- net SCL: track 0.00 -> 34.6 mm
- net SDA: track 5.08 -> 38.2 mm
- net SCK: track 0.00 -> 24.5 mm
- net CS: track 0.13 -> 18.4 mm
- net GND: track 19.9 -> 4.57 mm, vias 8 -> 1
- net Net-(D1-K): track 2.17 -> 7.02 mm, vias 0 -> 1
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- added copper zone on F.Cu, net +5V
- added copper zone on B.Cu, net GND
- removed copper zone on In1.Cu, net +5V
- removed copper zone on In2.Cu, net GND
Other:
- board size 45.1 x 68.6 mm -> 48.3 x 68.6 mm
- copper layers 4 -> 2

Commit message: fox v1
Parts:
- removed BZ1: Buzzer, Buzzer_Beeper:Buzzer_12x9.5RM7.6
- added J2: Conn_01x03, Connector_PinHeader_2.54mm:PinHeader_1x03_P2.54mm_Vertical, F.Cu at (68.6, 81.3)
- added J3: Conn_01x03, Connector_PinHeader_2.54mm:PinHeader_1x03_P2.54mm_Vertical, F.Cu at (65.0, 81.3)
- added J4: Conn_01x03, Connector_PinHeader_2.54mm:PinHeader_1x03_P2.54mm_Vertical, F.Cu at (61.5, 81.3)
- added J5: Conn_01x03, Connector_PinHeader_2.54mm:PinHeader_1x03_P2.54mm_Vertical, F.Cu at (57.9, 81.3)
- added J6: Conn_01x03, Connector_PinHeader_2.54mm:PinHeader_1x03_P2.54mm_Vertical, F.Cu at (73.2, 81.3)
- D1: footprint LED_THT:LED_D5.0mm-4_RGB -> LED_THT:LED_D5.0mm-4_RGB_Wide_Pins
- moved A2 13.7 mm to (55.1, 34.3), turned to 90 degrees
- moved C9 13.3 mm to (56.4, 30.5), turned to 0 degrees
- moved D1 11.0 mm to (49.3, 24.6)
- moved U3 5.33 mm to (59.8, 76.2)
- moved A1 5.33 mm to (58.4, 46.2)
- moved C5 5.08 mm to (58.8, 71.1)
- moved R1 3.49 mm to (46.7, 33.0)
- moved C4 1.40 mm to (29.8, 33.5)
- moved C2 0.89 mm to (59.7, 49.8)
- moved U2 0.87 mm to (40.6, 27.9)
- moved J1 0.85 mm to (31.0, 29.0)
- moved C1 0.63 mm to (29.8, 38.1)
- moved C8 0.11 mm to (45.2, 21.0)
Connections:
- U1 pad 10: INTNRF -> servoout2
- U1 pad 12: greenled -> servoout3
- U1 pad 15: redled -> servoout4
- U1 pad 5: unconnected-(U1-VDET_1/GPIO34/ADC1_CH6-Pad5) -> INTMPU
- U1 pad 6: unconnected-(U1-VDET_2/GPIO35/ADC1_CH7-Pad6) -> INTNRF
- U1 pad 7: unconnected-(U1-32K_XP/GPIO32/ADC1_CH4-Pad7) -> greenled
- U1 pad 8: buzzer -> redled
- U1 pad 9: INTMPU -> servoout1
Routing:
- net servoout1: track 0.00 -> 49.3 mm
- net servoout2: track 0.00 -> 44.3 mm
- net buzzer: track 40.9 -> 0.00 mm
- net SDA: track 38.2 -> 78.6 mm
- net servoout3: track 0.00 -> 37.9 mm
- net SCL: track 34.6 -> 70.1 mm, vias 0 -> 2
- net servoout4: track 0.00 -> 31.2 mm
- net MOSI: track 60.8 -> 34.4 mm, vias 0 -> 2
- net blueled: track 53.2 -> 71.5 mm, vias 2 -> 3
- net greenled: track 54.0 -> 39.2 mm
- net redled: track 56.4 -> 44.7 mm, vias 3 -> 2
- net +5V: track 18.2 -> 29.5 mm, vias 1 -> 4
- net INTMPU: track 41.0 -> 51.8 mm
- net MISO: track 40.2 -> 31.9 mm
- net SCK: track 24.5 -> 31.4 mm, vias 0 -> 2
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
Commit message: FLIGHT Compupdate
Parts:
- removed C9: 1uf, Capacitor_SMD:C_0805_2012Metric_Pad1.18x1.45mm_HandSolder
- removed U3: NRF24L01_Breakout, RF_Module:nRF24L01_Breakout
- added BZ1: Buzzer, Buzzer_Beeper:Buzzer_12x9.5RM7.6, F.Cu at (58.2, 27.4)
- moved C6 45.9 mm to (67.6, 56.9), turned to 90 degrees
- moved C2 44.0 mm to (32.5, 84.3)
- moved A1 30.7 mm to (70.6, 74.4), turned to 180 degrees
- moved A2 28.6 mm to (70.9, 58.2), turned to 180 degrees
- moved C5 9.47 mm to (68.1, 73.2), turned to 90 degrees
- moved U1 2.76 mm to (28.6, 38.5)
- moved C1 2.03 mm to (29.8, 36.1)
- moved C3 1.91 mm to (32.4, 81.3)
- moved D1 1.78 mm to (49.3, 22.9)
Connections:
- A1 pad 1: +5V -> +3V3
- A2 pad 1: +5V -> +3V3
- C5 pad 1: +5V -> +3V3
- C6 pad 1: +5V -> +3V3
- U1 pad 11: CE -> unconnected-(U1-ADC2_CH7/GPIO27-Pad11)
- U1 pad 29: CS -> unconnected-(U1-*GPIO5-Pad29)
- U1 pad 30: SCK -> unconnected-(U1-GPIO18-Pad30)
- U1 pad 31: MISO -> unconnected-(U1-GPIO19-Pad31)
- U1 pad 6: INTNRF -> buzzer
Routing:
- net +5V: track 29.5 -> 123.0 mm, vias 4 -> 1
- net INTNRF: track 47.0 -> 0.00 mm
- net buzzer: track 0.00 -> 45.4 mm, vias 0 -> 2
- net CE: track 40.7 -> 0.00 mm
- net MOSI: track 34.4 -> 0.00 mm, vias 2 -> 0
- net MISO: track 31.9 -> 0.00 mm
- net SCK: track 31.4 -> 0.00 mm, vias 2 -> 0
- net SDA: track 78.6 -> 54.3 mm, vias 0 -> 1
- net blueled: track 71.5 -> 55.7 mm, vias 3 -> 0
- net CS: track 13.9 -> 0.00 mm
- net SCL: track 70.1 -> 59.5 mm, vias 2 -> 0
- net redled: track 44.7 -> 37.9 mm, vias 2 -> 0
- net GND: track 3.65 -> 9.12 mm, vias 0 -> 4
- net INTMPU: track 51.8 -> 48.4 mm
- net Net-(D1-K): track 2.54 -> 4.32 mm
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- added copper zone on F.Cu, net +3V3
- removed copper zone on F.Cu, net +5V

Commit message: lots of stuff
Parts:
- added J7: Screw_Terminal_01x02, TerminalBlock:TerminalBlock_bornier-2_P5.08mm, F.Cu at (70.5, 30.5)
- added J8: Screw_Terminal_01x02, TerminalBlock:TerminalBlock_bornier-2_P5.08mm, F.Cu at (70.5, 41.3)
- added Q1: IRF540N, Package_TO_SOT_THT:TO-220-3_Vertical, F.Cu at (64.8, 41.3)
- added Q2: IRF540N, Package_TO_SOT_THT:TO-220-3_Vertical, F.Cu at (59.7, 41.3)
- moved J6 31.8 mm to (73.7, 49.5)
- moved C8 13.5 mm to (35.6, 30.5)
- moved A1 12.3 mm to (58.4, 75.7), turned to 90 degrees
- moved U2 11.8 mm to (28.9, 26.0), turned to -90 degrees
- moved C6 9.43 mm to (69.8, 66.0), turned to 180 degrees
- moved J1 9.02 mm to (36.2, 21.6), turned to 0 degrees
- moved C5 8.38 mm to (59.7, 73.0), turned to 0 degrees
- moved C7 5.85 mm to (33.0, 27.3)
- moved C2 5.59 mm to (32.4, 78.7)
- moved A2 5.43 mm to (69.8, 63.5)
- moved R1 3.30 mm to (47.6, 29.8)
- moved BZ1 3.24 mm to (55.3, 26.0)
- moved U1 3.17 mm to (28.6, 35.3)
- moved D1 2.17 mm to (49.5, 20.7)
- moved C1 1.91 mm to (31.8, 36.1)
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Connections:
- U1 pad 30: unconnected-(U1-GPIO18-Pad30) -> pyro1
- U1 pad 31: unconnected-(U1-GPIO19-Pad31) -> pyro2
Routing:
- net +BATT: track 16.0 -> 59.1 mm
- net SDA: track 54.3 -> 81.8 mm
- net SCL: track 59.5 -> 80.7 mm, vias 0 -> 2
- net pyro2out: track 0.00 -> 19.2 mm
- net pyro1: track 0.00 -> 18.9 mm, vias 0 -> 1
- net pyro2: track 0.00 -> 14.2 mm, vias 0 -> 1
- net pyro1out: track 0.00 -> 6.77 mm
- net INTMPU: track 48.4 -> 54.2 mm
- net +5V: track 123.0 -> 118.7 mm
- net +3V3: track 6.03 -> 10.1 mm
- net servoout4: track 32.3 -> 35.9 mm
- net GND: track 9.12 -> 5.66 mm
- net servoout2: track 44.7 -> 47.7 mm
- net servoout1: track 49.3 -> 52.2 mm, vias 0 -> 1
- net Net-(D1-K): track 4.32 -> 3.04 mm
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Other:
- board size 48.3 x 68.6 mm -> 48.9 x 71.1 mm

Commit message: stuff
Parts:
- removed J6: Conn_01x03, Connector_PinHeader_2.54mm:PinHeader_1x03_P2.54mm_Vertical
Connections:
- A1 pad 5: unconnected-(A1-CSB-Pad5) -> +3V3
- A1 pad 6: unconnected-(A1-SD0-Pad6) -> GND
Routing:
- net SCL: track 80.7 -> 61.5 mm
- net SDA: track 81.8 -> 74.4 mm
