File: avionics/hyades/hyades/hyades.kicad_pcb (KiCad board)
At the start: 4 copper layers, 84 x 28 mm, 69 parts, among them J1 USB_B_Micro, J10 AXK5S30347YG, J12 AXK5S30347YG, J13 AXK5S30347YG, J14 AXK5S30347YG, J15 AXK5S30347YG, J16 AXK5S30347YG, J9 MEM2067-02-180-00-A, Q1 AO3401A, Q2 Q_NMOS_GSD, Q3 Q_NMOS_GSD, SW1 SW_MEC_5E, U1 LM317_SOT-223, U2 LM317_SOT-223, U3 USBLC6-2SC6, U4 BMI088, U5 BMP390L, U6 W25Q32JVSS, U7 STM32F405RGTx, X1 ECS-2520MV-xxx-xx

Commit message: stuff
Parts:
- moved X1 86.8 mm to (109.2, 105.7), turned to 180 degrees
Changed lines of the file:
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@@
   )
   (footprint "Oscillator:Oscillator_SMD_ECS_2520MV-xxx-xx-4Pin_2.5x2.0mm" (layer "F.Cu")
-    (at 175.45 49.63)
+    (at 109.22 105.664 180)
     (descr "Miniature Crystal Clock Oscillator ECS 2520MV series, https://www.ecsxtal.com/store/pdf/ECS-2520MV.pdf")
     (tags "Miniature Crystal Clock Oscillator ECS 2520MV series SMD SMT HCMOS")
@@
     (fp_line (start 1 -1.25) (end 1 1.25)
       (stroke (width 0.1) (type solid)) (layer "F.Fab"))
-    (pad "1" smd roundrect (at -0.725 -0.925) (size 0.8 0.9) (layers "F.Cu" "F.Paste" "F.Mask") (roundrect_rratio 0.25)
+    (pad "1" smd roundrect (at -0.725 -0.925 180) (size 0.8 0.9) (layers "F.Cu" "F.Paste" "F.Mask") (roundrect_rratio 0.25)
       (net 6 "+3.3VA") (pinfunction "Tri-State") (pintype "input"))
-    (pad "2" smd roundrect (at -0.725 0.925) (size 0.8 0.9) (layers "F.Cu" "F.Paste" "F.Mask") (roundrect_rratio 0.25)
+    (pad "2" smd roundrect (at -0.725 0.925 180) (size 0.8 0.9) (layers "F.Cu" "F.Paste" "F.Mask") (roundrect_rratio 0.25)
       (net 2 "GND") (pinfunction "GND") (pintype "power_in"))
-    (pad "3" smd roundrect (at 0.725 0.925) (size 0.8 0.9) (layers "F.Cu" "F.Paste" "F.Mask") (roundrect_rratio 0.25)
+    (pad "3" smd roundrect (at 0.725 0.925 180) (size 0.8 0.9) (layers "F.Cu" "F.Paste" "F.Mask") (roundrect_rratio 0.25)
       (net 61 "OSCIN") (pinfunction "OUT") (pintype "output"))
-    (pad "4" smd roundrect (at 0.725 -0.925) (size 0.8 0.9) (layers "F.Cu" "F.Paste" "F.Mask") (roundrect_rratio 0.25)
+    (pad "4" smd roundrect (at 0.725 -0.925 180) (size 0.8 0.9) (layers "F.Cu" "F.Paste" "F.Mask") (roundrect_rratio 0.25)
       (net 6 "+3.3VA") (pinfunction "VDD") (pintype "power_in"))
     (model "${KICAD6_3DMODEL_DIR}/Oscillator.3dshapes/Oscillator_SMD_ECS_2520MV-xxx-xx-4Pin_2.5x2.0mm.wrl"

Commit message: more avionics work
Parts:
- added C12: 100nf, Capacitor_SMD:C_0603_1608Metric, F.Cu at (247.2, 52.0)
- added C13: 100nf, Capacitor_SMD:C_0603_1608Metric, F.Cu at (247.2, 54.5)
- added C14: 100nf, Capacitor_SMD:C_0603_1608Metric, F.Cu at (247.2, 57.0)
- added C15: 100nf, Capacitor_SMD:C_0603_1608Metric, F.Cu at (247.2, 59.5)
- added C16: 100nf, Capacitor_SMD:C_0603_1608Metric, F.Cu at (247.2, 62.0)
- added C20: 100uf, Capacitor_SMD:C_0805_2012Metric, F.Cu at (243.1, 80.0)
- added C27: 100nf, Capacitor_SMD:C_0603_1608Metric, F.Cu at (247.2, 64.5)
- added C30: 100uf, Capacitor_SMD:C_0805_2012Metric, F.Cu at (243.1, 83.0)
- added C31: 100uf, Capacitor_SMD:C_0805_2012Metric, F.Cu at (243.1, 86.0)
- added C32: 100uf, Capacitor_SMD:C_0805_2012Metric, F.Cu at (243.1, 89.0)
- added H1: MountingHole_Pad, MountingHole:MountingHole_2.2mm_M2_Pad, F.Cu at (112.8, 93.1)
- added H10: MountingHole_Pad, MountingHole:MountingHole_2.2mm_M2_Pad, F.Cu at (168.2, 93.1)
- added H11: MountingHole_Pad, MountingHole:MountingHole_2.2mm_M2_Pad, F.Cu at (186.2, 93.1)
- added H12: MountingHole_Pad, MountingHole:MountingHole_2.2mm_M2_Pad, F.Cu at (186.2, 111.1)
- added H2: MountingHole_Pad, MountingHole:MountingHole_2.2mm_M2_Pad, F.Cu at (130.2, 111.1)
- added H3: MountingHole_Pad, MountingHole:MountingHole_2.2mm_M2_Pad, F.Cu at (112.2, 110.6)
- added H4: MountingHole_Pad, MountingHole:MountingHole_2.2mm_M2_Pad, F.Cu at (130.2, 93.1)
- added H5: MountingHole_Pad, MountingHole:MountingHole_2.2mm_M2_Pad, F.Cu at (140.2, 93.1)
- added H6: MountingHole_Pad, MountingHole:MountingHole_2.2mm_M2_Pad, F.Cu at (158.2, 93.1)
- added H7: MountingHole_Pad, MountingHole:MountingHole_2.2mm_M2_Pad, F.Cu at (140.2, 111.1)
- added H8: MountingHole_Pad, MountingHole:MountingHole_2.2mm_M2_Pad, F.Cu at (158.2, 111.1)
- added H9: MountingHole_Pad, MountingHole:MountingHole_2.2mm_M2_Pad, F.Cu at (168.2, 111.1)
- added J11: Switch Terminal, TerminalBlock:TerminalBlock_bornier-2_P5.08mm, F.Cu at (236.9, 64.3)
- added J17: Conn_02x04_Odd_Even, Connector_PinHeader_2.54mm:PinHeader_2x04_P2.54mm_Vertical, F.Cu at (236.0, 80.8)
- added J18: SPI HEADER, Connector_PinHeader_2.54mm:PinHeader_2x03_P2.54mm_Vertical, F.Cu at (214.1, 109.1)
- added J19: I2C HEADER, Connector_PinHeader_2.54mm:PinHeader_1x03_P2.54mm_Vertical, F.Cu at (223.2, 108.1)
- added J2: Servo1, Connector_PinHeader_2.54mm:PinHeader_1x03_P2.54mm_Vertical, F.Cu at (236.0, 71.1)
- added J20: UART HEADER, Connector_PinHeader_2.54mm:PinHeader_1x03_P2.54mm_Vertical, F.Cu at (227.8, 108.1)
- added J3: Servo2, Connector_PinHeader_2.54mm:PinHeader_1x03_P2.54mm_Vertical, F.Cu at (240.6, 71.1)
- added J4: Servo3, Connector_PinHeader_2.54mm:PinHeader_1x03_P2.54mm_Vertical, F.Cu at (245.3, 71.1)
- added J5: Servo4, Connector_PinHeader_2.54mm:PinHeader_1x03_P2.54mm_Vertical, F.Cu at (249.9, 71.1)
- added J6: Screw_Terminal_01x04, TerminalBlock:TerminalBlock_bornier-4_P5.08mm, F.Cu at (205.1, 79.1)
- added J7: Screw_Terminal_01x04, TerminalBlock:TerminalBlock_bornier-4_P5.08mm, F.Cu at (205.1, 88.1)
- added J8: Batt Terminal, TerminalBlock:TerminalBlock_bornier-2_P5.08mm, F.Cu at (236.9, 55.2)
- added JP1: Servo Power, Jumper:SolderJumper-3_P1.3mm_Bridged12_RoundedPad1.0x1.5mm, F.Cu at (226.4, 76.3)
- added JP2: I2C POWER, Jumper:SolderJumper-3_P1.3mm_Bridged12_RoundedPad1.0x1.5mm, F.Cu at (226.4, 80.2)
- added JP3: UART POWER, Jumper:SolderJumper-3_P1.3mm_Bridged12_RoundedPad1.0x1.5mm, F.Cu at (226.4, 84.0)
- added JP5: SPI Power, Jumper:SolderJumper-3_P1.3mm_Bridged12_RoundedPad1.0x1.5mm, F.Cu at (226.4, 87.8)
- added R7: 470, Resistor_SMD:R_0603_1608Metric, F.Cu at (247.2, 67.0)
- F1: value 1a -> 2a
- J10, J16: value AXK5S30347YG -> BOARDTOBOARDB
- J12, J13: value AXK5S30347YG -> BOARDTOBOARDF
- J14: value AXK5S30347YG -> BOARDTOBOARDF; moved to F.Cu
- J15: value AXK5S30347YG -> BOARDTOBOARDB; moved to B.Cu
- U3, X1: moved to B.Cu
- moved U3 54.7 mm to (121.8, 106.9), turned to 90 degrees
- moved J14 28.0 mm to (177.2, 92.1)
- moved J15 28.0 mm to (149.2, 92.1)
- moved X1 13.9 mm to (122.3, 100.8), turned to 0 degrees
- moved U6 13.6 mm to (149.7, 113.2), turned to 0 degrees
- moved J9 4.38 mm to (149.2, 107.5)
- moved J1 0.62 mm to (121.6, 113.2)
- turned J16 to 0 degrees
- turned U7 to -90 degrees
Connections:
- J10 pad 2: +3V3 -> PC8
- J12 pad 1: +3V3 -> PC8
- J12 pad 10: +12P -> SDA
- J12 pad 11: SCL -> FLASH CS
- J12 pad 12: FLASH CS -> SCL
- J12 pad 13: SERVO1 -> CS SD
- J12 pad 14: CS SD -> SERVO1
- J12 pad 15: SERVO2 -> ACCEL INT2
- J12 pad 16: ACCEL INT2 -> SERVO2
- J12 pad 17: SERVO3 -> ACCEL INT1
- J12 pad 18: ACCEL INT1 -> SERVO3
- J12 pad 19: SERVO4 -> GYRO INT3
- J12 pad 20: GYRO INT3 -> SERVO4
- J12 pad 21: SCK -> GYRO INT4
- J12 pad 22: GYRO INT4 -> SCK
- J12 pad 23: MISO -> BARO INT
- J12 pad 24: BARO INT -> MISO
- J12 pad 25: MOSI -> P1 EN
- J12 pad 26: P1 EN -> MOSI
- J12 pad 27: PB14 -> P2 EN
- J12 pad 28: P2 EN -> PB14
- J12 pad 3: USART2 TX -> +5V
- J12 pad 4: +5V -> USART2 TX
- J12 pad 5: USART2 RX -> +5V
- J12 pad 6: +5V -> USART2 RX
- J12 pad 7: PB15 -> +12P
- J12 pad 8: +12P -> PB15
- J12 pad 9: SDA -> +12P
- J13 pad 1: +3V3 -> PC8
- J13 pad 10: +12P -> SDA
- J13 pad 11: SCL -> FLASH CS
- J13 pad 12: FLASH CS -> SCL
- J13 pad 13: SERVO1 -> CS SD
- J13 pad 14: CS SD -> SERVO1
- J13 pad 15: SERVO2 -> ACCEL INT2
- J13 pad 16: ACCEL INT2 -> SERVO2
- J13 pad 17: SERVO3 -> ACCEL INT1
- J13 pad 18: ACCEL INT1 -> SERVO3
- J13 pad 19: SERVO4 -> GYRO INT3
- J13 pad 20: GYRO INT3 -> SERVO4
- J13 pad 21: SCK -> GYRO INT4
- J13 pad 22: GYRO INT4 -> SCK
- J13 pad 23: MISO -> BARO INT
- J13 pad 24: BARO INT -> MISO
- J13 pad 25: MOSI -> P1 EN
- J13 pad 26: P1 EN -> MOSI
- J13 pad 27: PB14 -> P2 EN
- J13 pad 28: P2 EN -> PB14
- J13 pad 3: USART2 TX -> +5V
- J13 pad 4: +5V -> USART2 TX
- J13 pad 5: USART2 RX -> +5V
- J13 pad 6: +5V -> USART2 RX
- J13 pad 7: PB15 -> +12P
- J13 pad 8: +12P -> PB15
- J13 pad 9: SDA -> +12P
- J14 pad 1: +3V3 -> PC8
- J14 pad 10: +12P -> SDA
- J14 pad 11: SCL -> FLASH CS
- J14 pad 12: FLASH CS -> SCL
- J14 pad 13: SERVO1 -> CS SD
- J14 pad 14: CS SD -> SERVO1
- J14 pad 15: SERVO2 -> ACCEL INT2
- J14 pad 16: ACCEL INT2 -> SERVO2
- J14 pad 17: SERVO3 -> ACCEL INT1
- J14 pad 18: ACCEL INT1 -> SERVO3
- J14 pad 19: SERVO4 -> GYRO INT3
- J14 pad 20: GYRO INT3 -> SERVO4
- J14 pad 21: SCK -> GYRO INT4
- J14 pad 22: GYRO INT4 -> SCK
- J14 pad 23: MISO -> BARO INT
- J14 pad 24: BARO INT -> MISO
- J14 pad 25: MOSI -> P1 EN
- J14 pad 26: P1 EN -> MOSI
- J14 pad 27: PB14 -> P2 EN
- J14 pad 28: P2 EN -> PB14
- J14 pad 3: USART2 TX -> +5V
- J14 pad 4: +5V -> USART2 TX
- J14 pad 5: USART2 RX -> +5V
- J14 pad 6: +5V -> USART2 RX
- J14 pad 7: PB15 -> +12P
- J14 pad 8: +12P -> PB15
- J14 pad 9: SDA -> +12P
- J15 pad 2: +3V3 -> PC8
- J16 pad 2: +3V3 -> PC8
- U7 pad 39: unconnected-(U7-PC8-Pad39) -> PC8
Routing:
- net GND: vias 0 -> 48
- added copper zone on In1.Cu, net +3V3
- added copper zone on In2.Cu, net GND

Commit message: bunch of stuff
Parts:
- removed C21, C22, C23, C24, C25, C26: 1uf, Capacitor_SMD:C_0805_2012Metric
- removed C30, C31, C32: 100uf, Capacitor_SMD:C_0805_2012Metric
- removed D1: D_Small, Diode_SMD:D_0805_2012Metric
- added D6: LED, LED_SMD:LED_0805_2012Metric, F.Cu at (102.4, 105.4)
- added H13: MountingHole_Pad, MountingHole:MountingHole_2.2mm_M2_Pad, F.Cu at (84.2, 93.1)
- added H14: MountingHole_Pad, MountingHole:MountingHole_2.2mm_M2_Pad, F.Cu at (102.2, 93.1)
- added H15: MountingHole_Pad, MountingHole:MountingHole_2.2mm_M2_Pad, F.Cu at (102.2, 111.1)
- added H16: MountingHole_Pad, MountingHole:MountingHole_2.2mm_M2_Pad, F.Cu at (84.2, 111.1)
- added R19: 470, Resistor_SMD:R_0603_1608Metric, F.Cu at (102.4, 107.2)
- added TP1: Connector, TestPoint:TestPoint_Keystone_5019_Minature, F.Cu at (82.1, 100.7)
- added TP2: Connector, TestPoint:TestPoint_Keystone_5019_Minature, F.Cu at (82.0, 97.7)
- added TP3: Connector, TestPoint:TestPoint_Keystone_5019_Minature, F.Cu at (82.0, 103.6)
- added TP4: Connector, TestPoint:TestPoint_Keystone_5019_Minature, F.Cu at (82.0, 106.6)
- C12, C16, C20, F1, F2, FB1, J10, JP2, JP5, Q1, R1, R2, R3, R4, R5, R6, SW1: moved to B.Cu
- C28: footprint Capacitor_SMD:C_0805_2012Metric -> Capacitor_SMD:C_0603_1608Metric
- C29: value 1uf -> 2u2; footprint Capacitor_SMD:C_0805_2012Metric -> Capacitor_SMD:C_0603_1608Metric
- J11: value Switch Terminal -> BOARDTOBOARDF; footprint TerminalBlock:TerminalBlock_bornier-2_P5.08mm -> SamacSys_Parts:AXK5S30347YG
- J12, U6, X1: moved to F.Cu
- J19, J20: footprint Connector_PinHeader_2.54mm:PinHeader_1x03_P2.54mm_Vertical -> Connector_PinHeader_2.54mm:PinHeader_1x04_P2.54mm_Vertical
- J6: value Screw_Terminal_01x04 -> Screw_Terminal_01x02; footprint TerminalBlock:TerminalBlock_bornier-4_P5.08mm -> TerminalBlock_TE-Connectivity:TerminalBlock_TE_282834-2_1x02_P2.54mm_Horizontal
- J7: footprint TerminalBlock:TerminalBlock_bornier-4_P5.08mm -> TerminalBlock_TE-Connectivity:TerminalBlock_TE_282834-4_1x04_P2.54mm_Horizontal
- J8: value Batt Terminal -> BOARDTOBOARDB; footprint TerminalBlock:TerminalBlock_bornier-2_P5.08mm -> SamacSys_Parts:AXK5S30347YG; moved to B.Cu
- moved J8 148.3 mm to (93.2, 92.1)
- moved J11 146.3 mm to (93.2, 92.1)
- moved C27 142.6 mm to (119.8, 128.6)
- moved C13 140.5 mm to (118.5, 110.9)
- moved C15 139.6 mm to (113.3, 99.0)
- moved C16 134.4 mm to (118.2, 99.7), turned to 180 degrees
- moved C14 133.3 mm to (125.6, 111.6), turned to 90 degrees
- moved C12 131.0 mm to (125.2, 99.6)
- moved R13 116.2 mm to (214.3, 112.0)
- moved R14 116.2 mm to (214.3, 114.5)
- moved R17 112.1 mm to (214.8, 101.3)
- moved R18 112.1 mm to (214.8, 103.8)
- moved R5 106.4 mm to (95.5, 110.5), turned to 180 degrees
- moved R11 104.3 mm to (154.6, 139.3)
- moved R3 103.6 mm to (95.1, 100.9)
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Connections:
- J11 pad 1: +BATT -> PC8
- J11 pad 2: TOGGLED12V -> +3V3
- J17 pad 3: unconnected-(J17-Pin_3-Pad3) -> +12P
- J17 pad 5: +12P -> GND
- J17 pad 6: unconnected-(J17-Pin_6-Pad6) -> +3V3
- J6 pad 1: GND -> +12P
- J6 pad 2: +3V3 -> ARM+
- J8 pad 1: +BATT -> +3V3
- J8 pad 2: GND -> PC8
- JP2 pad 1: +5V -> +3V3
- JP2 pad 3: +3V3 -> +5V
- JP3 pad 1: +5V -> +3V3
- JP3 pad 3: +3V3 -> +5V
- JP5 pad 1: +5V -> +3V3
- JP5 pad 3: +3V3 -> +5V
- R10 pad 1: +12V -> +12P
Routing:
- net GND: track 0.00 -> 27.5 mm, vias 48 -> 70
- net +3V3: track 0.00 -> 8.09 mm, vias 0 -> 7
- net SERVOPOWER: track 0.00 -> 7.77 mm
- net +12P: track 0.00 -> 5.77 mm
- net TOGGLED12V: track 0.00 -> 3.59 mm, vias 0 -> 1
- net +BATT: track 0.00 -> 3.07 mm
- net Net-(U7-VCAP_2): track 0.00 -> 2.71 mm
- net +3.3VA: track 0.00 -> 2.69 mm
- net Net-(Q1-D): track 0.00 -> 2.69 mm
- net Net-(F2-Pad2): track 0.00 -> 2.49 mm
- net Net-(U7-VCAP_1): track 0.00 -> 2.11 mm
- net Net-(D6-A): track 0.00 -> 1.88 mm
- net Net-(D4-A): track 0.00 -> 1.84 mm
- net Net-(R3-Pad2): track 0.00 -> 1.56 mm
Other:
- board size 84 x 28 mm -> 112 x 28 mm
