File: avionics/hyades/hyades/hyades.kicad_sch (KiCad schematic)
At the start: 99 parts, among them J1 USB_B_Micro, J10 AXK5S30347YG, J11 Switch Terminal, J12 AXK5S30347YG, J13 AXK5S30347YG, J14 AXK5S30347YG, J15 AXK5S30347YG, J16 AXK5S30347YG, J2 Servo1, J3 Servo2, J4 Servo3, J5 Servo4, J6 Screw_Terminal_01x04, J7 Screw_Terminal_01x04, J8 Batt Terminal, J9 MEM2067-02-180-00-A, Q1 AO3401A, Q2 Q_NMOS_GSD, Q3 Q_NMOS_GSD, SW1 SW_MEC_5E, SW2 SW_SPDT, U1 LM317_SOT-223, U2 LM317_SOT-223, U3 USBLC6-2SC6, U4 BMI088, U5 BMP390L, U6 W25Q32JVSS, U7 STM32F405RGTx, X1 ECS-2520MV-xxx-xx

Commit message: stuff
Parts:
- C12, C13, C14, C15, C16, C27: footprint (none) -> Capacitor_SMD:C_0603_1608Metric
- C20: footprint (none) -> Capacitor_SMD:C_0805_2012Metric
- H1, H10, H11, H12, H2, H3, H4, H5, H6, H7, H8, H9: footprint (none) -> MountingHole:MountingHole_3.2mm_M3_Pad
- J11, J8: footprint (none) -> TerminalBlock:TerminalBlock_bornier-2_P5.08mm
- J2, J3, J4, J5: footprint (none) -> Connector_PinHeader_2.54mm:PinHeader_1x03_P2.54mm_Vertical
- J6, J7: footprint (none) -> TerminalBlock:TerminalBlock_bornier-4_P5.08mm
- JP1: footprint (none) -> Jumper:SolderJumper-3_P1.3mm_Bridged12_RoundedPad1.0x1.5mm
- R7: footprint (none) -> Resistor_SMD:R_0603_1608Metric
Changed lines of the file:
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@@
       (effects (font (size 1.27 1.27)) (justify left))
     )
-    (property "Footprint" "" (at 385.445 329.565 0)
+    (property "Footprint" "TerminalBlock:TerminalBlock_bornier-2_P5.08mm" (at 385.445 329.565 0)
       (effects (font (size 1.27 1.27)) hide)
     )
@@
       (effects (font (size 1.27 1.27)) (justify left))
     )
-    (property "Footprint" "" (at 93.345 46.355 0)
+    (property "Footprint" "TerminalBlock:TerminalBlock_bornier-4_P5.08mm" (at 93.345 46.355 0)
       (effects (font (size 1.27 1.27)) hide)
     )
@@
       (effects (font (size 1.27 1.27)) (justify left))
     )
-    (property "Footprint" "" (at 545.465 287.02 0)
+    (property "Footprint" "MountingHole:MountingHole_3.2mm_M3_Pad" (at 545.465 287.02 0)
       (effects (font (size 1.27 1.27)) hide)
     )
@@
       (effects (font (size 1.27 1.27)) (justify left))
     )
-    (property "Footprint" "" (at 198.755 53.975 0)
+    (property "Footprint" "MountingHole:MountingHole_3.2mm_M3_Pad" (at 198.755 53.975 0)
       (effects (font (size 1.27 1.27)) hide)
     )
@@
       (effects (font (size 1.27 1.27)) (justify left))
     )
-    (property "Footprint" "" (at 545.465 276.86 0)
+    (property "Footprint" "MountingHole:MountingHole_3.2mm_M3_Pad" (at 545.465 276.86 0)
       (effects (font (size 1.27 1.27)) hide)
     )
@@
       (effects (font (size 1.27 1.27)) (justify left))
     )
-    (property "Footprint" "" (at 198.755 48.895 0)
+    (property "Footprint" "MountingHole:MountingHole_3.2mm_M3_Pad" (at 198.755 48.895 0)
       (effects (font (size 1.27 1.27)) hide)
     )
@@
       (effects (font (size 1.27 1.27)) (justify right))
     )
-    (property "Footprint" "" (at 511.175 243.84 0)
+    (property "Footprint" "Capacitor_SMD:C_0603_1608Metric" (at 511.175 243.84 0)
       (effects (font (size 1.27 1.27)) hide)
     )
@@
       (effects (font (size 1.27 1.27)) (justify left))
     )
-    (property "Footprint" "" (at 388.62 127 0)
+    (property "Footprint" "MountingHole:MountingHole_3.2mm_M3_Pad" (at 388.62 127 0)
       (effects (font (size 1.27 1.27)) hide)
     )
@@
       (effects (font (size 1.27 1.27)) (justify right))
     )
-    (property "Footprint" "" (at 530.86 243.84 0)
+    (property "Footprint" "Capacitor_SMD:C_0603_1608Metric" (at 530.86 243.84 0)
       (effects (font (size 1.27 1.27)) hide)
     )
@@
       (effects (font (size 1.27 1.27)) (justify right))
     )
-    (property "Footprint" "" (at 30.48 30.48 0)
+    (property "Footprint" "Capacitor_SMD:C_0805_2012Metric" (at 30.48 30.48 0)
       (effects (font (size 1.27 1.27)) hide)
     )
@@
       (effects (font (size 1.27 1.27)) (justify left))
     )
-    (property "Footprint" "" (at 57.15 57.15 0)
+    (property "Footprint" "Connector_PinHeader_2.54mm:PinHeader_1x03_P2.54mm_Vertical" (at 57.15 57.15 0)
       (effects (font (size 1.27 1.27)) hide)
     )
@@
       (effects (font (size 1.27 1.27)) (justify left))
     )
-    (property "Footprint" "" (at 388.62 137.16 0)
+    (property "Footprint" "MountingHole:MountingHole_3.2mm_M3_Pad" (at 388.62 137.16 0)
       (effects (font (size 1.27 1.27)) hide)
     )
@@
       (effects (font (size 1.27 1.27)) (justify right))
     )
-    (property "Footprint" "" (at 541.02 243.84 0)
+    (property "Footprint" "Capacitor_SMD:C_0603_1608Metric" (at 541.02 243.84 0)
       (effects (font (size 1.27 1.27)) hide)
     )
@@
       (effects (font (size 1.27 1.27)) (justify left))
     )
-    (property "Footprint" "" (at 545.465 281.94 0)
+    (property "Footprint" "MountingHole:MountingHole_3.2mm_M3_Pad" (at 545.465 281.94 0)
       (effects (font (size 1.27 1.27)) hide)
     )
@@
       (effects (font (size 1.27 1.27)) (justify right))
     )
-    (property "Footprint" "" (at 560.705 243.84 0)
+    (property "Footprint" "Capacitor_SMD:C_0603_1608Metric" (at 560.705 243.84 0)
       (effects (font (size 1.27 1.27)) hide)
     )
@@
       (effects (font (size 1.27 1.27)) (justify left))
     )
-    (property "Footprint" "" (at 388.62 132.08 0)
+    (property "Footprint" "MountingHole:MountingHole_3.2mm_M3_Pad" (at 388.62 132.08 0)
       (effects (font (size 1.27 1.27)) hide)
     )
@@
       (effects (font (size 1.27 1.27)) (justify left))
     )
-    (property "Footprint" "" (at 36.83 26.67 0)
+    (property "Footprint" "Jumper:SolderJumper-3_P1.3mm_Bridged12_RoundedPad1.0x1.5mm" (at 36.83 26.67 0)
       (effects (font (size 1.27 1.27)) hide)
     )
@@
       (effects (font (size 1.27 1.27)) (justify left))
     )
-    (property "Footprint" "" (at 198.755 43.815 0)
+    (property "Footprint" "MountingHole:MountingHole_3.2mm_M3_Pad" (at 198.755 43.815 0)
       (effects (font (size 1.27 1.27)) hide)
     )
@@
       (effects (font (size 1.27 1.27)) (justify left))
     )
-    (property "Footprint" "" (at 476.885 262.89 0)
+    (property "Footprint" "Resistor_SMD:R_0603_1608Metric" (at 476.885 262.89 0)
       (effects (font (size 1.27 1.27)) hide)
     )
@@
       (effects (font (size 1.27 1.27)) (justify left))
     )
-    (property "Footprint" "" (at 545.465 292.1 0)
+    (property "Footprint" "MountingHole:MountingHole_3.2mm_M3_Pad" (at 545.465 292.1 0)
       (effects (font (size 1.27 1.27)) hide)
     )
@@
       (effects (font (size 1.27 1.27)) (justify left))
     )
-    (property "Footprint" "" (at 198.755 38.735 0)
+    (property "Footprint" "MountingHole:MountingHole_3.2mm_M3_Pad" (at 198.755 38.735 0)
       (effects (font (size 1.27 1.27)) hide)
     )
@@
       (effects (font (size 1.27 1.27)) (justify right))
     )
-    (property "Footprint" "" (at 551.18 243.84 0)
+    (property "Footprint" "Capacitor_SMD:C_0603_1608Metric" (at 551.18 243.84 0)
       (effects (font (size 1.27 1.27)) hide)
     )
@@
       (effects (font (size 1.27 1.27)) (justify right))
     )
-    (property "Footprint" "" (at 521.335 243.84 0)
+    (property "Footprint" "Capacitor_SMD:C_0603_1608Metric" (at 521.335 243.84 0)
       (effects (font (size 1.27 1.27)) hide)
     )
@@
       (effects (font (size 1.27 1.27)) (justify left))
     )
-    (property "Footprint" "" (at 385.445 339.09 0)
+    (property "Footprint" "TerminalBlock:TerminalBlock_bornier-2_P5.08mm" (at 385.445 339.09 0)
       (effects (font (size 1.27 1.27)) hide)
     )
@@
       (effects (font (size 1.27 1.27)) (justify left))
     )
-    (property "Footprint" "" (at 57.15 46.99 0)
+    (property "Footprint" "Connector_PinHeader_2.54mm:PinHeader_1x03_P2.54mm_Vertical" (at 57.15 46.99 0)
       (effects (font (size 1.27 1.27)) hide)
     )
@@
       (effects (font (size 1.27 1.27)) (justify left))
     )
-    (property "Footprint" "" (at 93.345 59.69 0)
+    (property "Footprint" "TerminalBlock:TerminalBlock_bornier-4_P5.08mm" (at 93.345 59.69 0)
       (effects (font (size 1.27 1.27)) hide)
     )
@@
       (effects (font (size 1.27 1.27)) (justify left))
     )
-    (property "Footprint" "" (at 57.15 77.47 0)
+    (property "Footprint" "Connector_PinHeader_2.54mm:PinHeader_1x03_P2.54mm_Vertical" (at 57.15 77.47 0)
       (effects (font (size 1.27 1.27)) hide)
     )
@@
       (effects (font (size 1.27 1.27)) (justify left))
     )
-    (property "Footprint" "" (at 57.15 67.31 0)
+    (property "Footprint" "Connector_PinHeader_2.54mm:PinHeader_1x03_P2.54mm_Vertical" (at 57.15 67.31 0)
       (effects (font (size 1.27 1.27)) hide)
     )
@@
       (effects (font (size 1.27 1.27)) (justify left))
     )
-    (property "Footprint" "" (at 388.62 142.24 0)
+    (property "Footprint" "MountingHole:MountingHole_3.2mm_M3_Pad" (at 388.62 142.24 0)
       (effects (font (size 1.27 1.27)) hide)
     )

Commit message: yhmm
Parts:
- added C30, C31, C32: 100uf, Capacitor_SMD:C_0805_2012Metric, symbol Device:C_Small
- added J17: Conn_02x04_Odd_Even, Connector_PinHeader_2.54mm:PinHeader_2x04_P2.54mm_Vertical, symbol Connector_Generic:Conn_02x04_Odd_Even
- added J18: SPI HEADER, symbol Connector_Generic:Conn_02x03_Top_Bottom
- added J19: I2C HEADER, symbol Connector_Generic:Conn_01x04
- added J20: UART HEADER, symbol Connector_Generic:Conn_01x04
- added JP2: I2C POWER, Jumper:SolderJumper-3_P1.3mm_Bridged12_RoundedPad1.0x1.5mm, symbol Jumper:SolderJumper_3_Open
- added JP3: UART POWER, Jumper:SolderJumper-3_P1.3mm_Bridged12_RoundedPad1.0x1.5mm, symbol Jumper:SolderJumper_3_Open
- added JP5: SPI Power, Jumper:SolderJumper-3_P1.3mm_Bridged12_RoundedPad1.0x1.5mm, symbol Jumper:SolderJumper_3_Open
- added SW3: SW_SPDT, symbol Switch:SW_SPDT
- F1: value 1a -> 2a
- J10, J15, J16: value AXK5S30347YG -> BOARDTOBOARDB
- J12, J13, J14: value AXK5S30347YG -> BOARDTOBOARDF
Connections:
- net +12P: now also J12.7, J12.9, J13.7, J13.9, J14.7, J14.9, J17.5 (Pin_5); no longer J12.10, J12.8, J13.10, J13.8, J14.10, J14.8
- net +3V3: now also J17.8 (Pin_8), JP2.3 (B), JP3.3 (B), JP5.3 (B), SW3.1 (A); no longer J10.2, J12.1, J13.1, J14.1, J15.2, J16.2
- net +5V: now also J12.3, J12.5, J13.3, J13.5, J14.3, J14.5, JP2.1 (A), JP3.1 (A), JP5.1 (A); no longer J12.4, J12.6, J13.4, J13.6, J14.4, J14.6
- net ACCEL INT1: now also J12.17, J13.17, J14.17; no longer J12.18, J13.18, J14.18
- net ACCEL INT2: now also J12.15, J13.15, J14.15; no longer J12.16, J13.16, J14.16
- net BARO INT: now also J12.23, J13.23, J14.23; no longer J12.24, J13.24, J14.24
- net BOOT0: now also SW3.2 (B)
- net CS SD: now also J12.13, J13.13, J14.13; no longer J12.14, J13.14, J14.14
- net FLASH CS: now also J12.11, J13.11, J14.11; no longer J12.12, J13.12, J14.12
- net GND: now also C30.1, C31.1, C32.1, J17.7 (Pin_7), J18.3 (Pin_3), J19.4 (Pin_4), J20.4 (Pin_4), SW3.3 (C)
- net GYRO INT3: now also J12.19, J13.19, J14.19; no longer J12.20, J13.20, J14.20
- net GYRO INT4: now also J12.21, J13.21, J14.21; no longer J12.22, J13.22, J14.22
- net MISO: now also J12.24, J13.24, J14.24, J18.5 (Pin_5); no longer J12.23, J13.23, J14.23
- net MOSI: now also J12.26, J13.26, J14.26, J18.6 (Pin_6); no longer J12.25, J13.25, J14.25
- net P1 EN: now also J12.25, J13.25, J14.25; no longer J12.26, J13.26, J14.26
- net P2 EN: now also J12.27, J13.27, J14.27; no longer J12.28, J13.28, J14.28
- net PB14: now also J12.28, J13.28, J14.28, J17.1 (Pin_1); no longer J12.27, J13.27, J14.27
- net PB15: now also J12.8, J13.8, J14.8, J17.2 (Pin_2); no longer J12.7, J13.7, J14.7
- net SCK: now also J12.22, J13.22, J14.22, J18.4 (Pin_4); no longer J12.21, J13.21, J14.21
- net SCL: now also J12.12, J13.12, J14.12, J19.3 (Pin_3); no longer J12.11, J13.11, J14.11
- net SDA: now also J12.10, J13.10, J14.10, J19.2 (Pin_2); no longer J12.9, J13.9, J14.9
- net SERVO1: now also J12.14, J13.14, J14.14; no longer J12.13, J13.13, J14.13
- net SERVO2: now also J12.16, J13.16, J14.16; no longer J12.15, J13.15, J14.15
- net SERVO3: now also J12.18, J13.18, J14.18; no longer J12.17, J13.17, J14.17
- net SERVO4: now also J12.20, J13.20, J14.20; no longer J12.19, J13.19, J14.19
- net USART2 RX: now also J12.6, J13.6, J14.6, J20.3 (Pin_3); no longer J12.5, J13.5, J14.5
- net USART2 TX: now also J12.4, J13.4, J14.4, J20.2 (Pin_2); no longer J12.3, J13.3, J14.3
- net PC8: now reaches U7.39 (PC8)
- net PC8: now also J10.2, J12.1, J13.1, J14.1, J15.2, J16.2, J18.2 (Pin_2)
- new net I2C POWER: C31.2, J19.1 (Pin_1), JP2.2 (C)
- new net SPI POWER: C30.2, J18.1 (Pin_1), JP5.2 (C)
- new net UART POWER: C32.2, J20.1 (Pin_1), JP3.2 (C)
Other:
- moved on the sheet: C1, C3, D1, F1, F2, FB1, H5, H6, H7, H8, J10, J11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

Commit message: more avionics work
Parts:
- H1, H10, H11, H12, H2, H3, H4, H5, H6, H7, H8, H9: footprint MountingHole:MountingHole_3.2mm_M3_Pad -> MountingHole:MountingHole_2.2mm_M2_Pad
- J18: footprint (none) -> Connector_PinHeader_2.54mm:PinHeader_2x03_P2.54mm_Vertical
- J19, J20: footprint (none) -> Connector_PinHeader_2.54mm:PinHeader_1x03_P2.54mm_Vertical
Changed lines of the file:
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@@
       (effects (font (size 1.27 1.27)) (justify left))
     )
-    (property "Footprint" "MountingHole:MountingHole_3.2mm_M3_Pad" (at 545.465 287.02 0)
+    (property "Footprint" "MountingHole:MountingHole_2.2mm_M2_Pad" (at 545.465 287.02 0)
       (effects (font (size 1.27 1.27)) hide)
     )
@@
       (effects (font (size 1.27 1.27)) (justify left))
     )
-    (property "Footprint" "MountingHole:MountingHole_3.2mm_M3_Pad" (at 198.755 53.975 0)
+    (property "Footprint" "MountingHole:MountingHole_2.2mm_M2_Pad" (at 198.755 53.975 0)
       (effects (font (size 1.27 1.27)) hide)
     )
@@
       (effects (font (size 1.27 1.27)) (justify left))
     )
-    (property "Footprint" "MountingHole:MountingHole_3.2mm_M3_Pad" (at 545.465 276.86 0)
+    (property "Footprint" "MountingHole:MountingHole_2.2mm_M2_Pad" (at 545.465 276.86 0)
       (effects (font (size 1.27 1.27)) hide)
     )
@@
       (effects (font (size 1.27 1.27)))
     )
-    (property "Footprint" "" (at 93.98 104.14 0)
+    (property "Footprint" "Connector_PinHeader_2.54mm:PinHeader_2x03_P2.54mm_Vertical" (at 93.98 104.14 0)
       (effects (font (size 1.27 1.27)) hide)
     )
@@
       (effects (font (size 1.27 1.27)) (justify left))
     )
-    (property "Footprint" "MountingHole:MountingHole_3.2mm_M3_Pad" (at 198.755 48.895 0)
+    (property "Footprint" "MountingHole:MountingHole_2.2mm_M2_Pad" (at 198.755 48.895 0)
       (effects (font (size 1.27 1.27)) hide)
     )
@@
       (effects (font (size 1.27 1.27)) (justify left))
     )
-    (property "Footprint" "MountingHole:MountingHole_3.2mm_M3_Pad" (at 392.43 127 0)
+    (property "Footprint" "MountingHole:MountingHole_2.2mm_M2_Pad" (at 392.43 127 0)
       (effects (font (size 1.27 1.27)) hide)
     )
@@
       (effects (font (size 1.27 1.27)) (justify left))
     )
-    (property "Footprint" "" (at 62.23 104.14 0)
+    (property "Footprint" "Connector_PinHeader_2.54mm:PinHeader_1x03_P2.54mm_Vertical" (at 62.23 104.14 0)
       (effects (font (size 1.27 1.27)) hide)
     )
@@
       (effects (font (size 1.27 1.27)) (justify left))
     )
-    (property "Footprint" "MountingHole:MountingHole_3.2mm_M3_Pad" (at 392.43 137.16 0)
+    (property "Footprint" "MountingHole:MountingHole_2.2mm_M2_Pad" (at 392.43 137.16 0)
       (effects (font (size 1.27 1.27)) hide)
     )
@@
       (effects (font (size 1.27 1.27)) (justify left))
     )
-    (property "Footprint" "MountingHole:MountingHole_3.2mm_M3_Pad" (at 545.465 281.94 0)
+    (property "Footprint" "MountingHole:MountingHole_2.2mm_M2_Pad" (at 545.465 281.94 0)
       (effects (font (size 1.27 1.27)) hide)
     )
@@
       (effects (font (size 1.27 1.27)) (justify left))
     )
-    (property "Footprint" "MountingHole:MountingHole_3.2mm_M3_Pad" (at 392.43 132.08 0)
+    (property "Footprint" "MountingHole:MountingHole_2.2mm_M2_Pad" (at 392.43 132.08 0)
       (effects (font (size 1.27 1.27)) hide)
     )
@@
       (effects (font (size 1.27 1.27)) (justify left))
     )
-    (property "Footprint" "MountingHole:MountingHole_3.2mm_M3_Pad" (at 198.755 43.815 0)
+    (property "Footprint" "MountingHole:MountingHole_2.2mm_M2_Pad" (at 198.755 43.815 0)
       (effects (font (size 1.27 1.27)) hide)
     )
@@
       (effects (font (size 1.27 1.27)) (justify left))
     )
-    (property "Footprint" "MountingHole:MountingHole_3.2mm_M3_Pad" (at 545.465 292.1 0)
+    (property "Footprint" "MountingHole:MountingHole_2.2mm_M2_Pad" (at 545.465 292.1 0)
       (effects (font (size 1.27 1.27)) hide)
     )
@@
       (effects (font (size 1.27 1.27)) (justify left))
     )
-    (property "Footprint" "MountingHole:MountingHole_3.2mm_M3_Pad" (at 198.755 38.735 0)
+    (property "Footprint" "MountingHole:MountingHole_2.2mm_M2_Pad" (at 198.755 38.735 0)
       (effects (font (size 1.27 1.27)) hide)
     )
@@
       (effects (font (size 1.27 1.27)) (justify left))
     )
-    (property "Footprint" "" (at 128.27 102.87 0)
+    (property "Footprint" "Connector_PinHeader_2.54mm:PinHeader_1x03_P2.54mm_Vertical" (at 128.27 102.87 0)
       (effects (font (size 1.27 1.27)) hide)
     )
@@
       (effects (font (size 1.27 1.27)) (justify left))
     )
-    (property "Footprint" "MountingHole:MountingHole_3.2mm_M3_Pad" (at 392.43 142.24 0)
+    (property "Footprint" "MountingHole:MountingHole_2.2mm_M2_Pad" (at 392.43 142.24 0)
       (effects (font (size 1.27 1.27)) hide)
     )

Commit message: bunch of stuff
Parts:
- removed C3 (x6): 1uf, Capacitor_SMD:C_0805_2012Metric, symbol Device:C_Small
- removed C30, C31, C32: 100uf, Capacitor_SMD:C_0805_2012Metric, symbol Device:C_Small
- removed D1: D_Small, Diode_SMD:D_0805_2012Metric, symbol Device:D_Small
- removed J11: Switch Terminal, TerminalBlock:TerminalBlock_bornier-2_P5.08mm, symbol Connector:Screw_Terminal_01x02
- removed J6: Screw_Terminal_01x04, TerminalBlock:TerminalBlock_bornier-4_P5.08mm, symbol Connector:Screw_Terminal_01x04
- removed J8: Batt Terminal, TerminalBlock:TerminalBlock_bornier-2_P5.08mm, symbol Connector:Screw_Terminal_01x02
- added D3: LED, LED_SMD:LED_0805_2012Metric, symbol Device:LED
- added H13, H14, H15, H16: MountingHole_Pad, MountingHole:MountingHole_2.2mm_M2_Pad, symbol Mechanical:MountingHole_Pad
- added J11: BOARDTOBOARDF, SamacSys_Parts:AXK5S30347YG, symbol SamacSys_Parts:AXK5S30347YG
- added J6: Screw_Terminal_01x02, TerminalBlock_TE-Connectivity:TerminalBlock_TE_282834-2_1x02_P2.54mm_Horizontal, symbol Connector:Screw_Terminal_01x02
- added J8: BOARDTOBOARDB, SamacSys_Parts:AXK5S30347YG, symbol SamacSys_Parts:AXK5S30347YG
- added R11: 470, Resistor_SMD:R_0603_1608Metric, symbol Device:R
- added TP1, TP2, TP3, TP4: Connector, TestPoint:TestPoint_Keystone_5019_Minature, symbol Connector:TestPoint
- C3: value 1uf -> 2u2; footprint Capacitor_SMD:C_0805_2012Metric -> Capacitor_SMD:C_0603_1608Metric
- C3: footprint Capacitor_SMD:C_0805_2012Metric -> Capacitor_SMD:C_0603_1608Metric
- J19, J20: footprint Connector_PinHeader_2.54mm:PinHeader_1x03_P2.54mm_Vertical -> Connector_PinHeader_2.54mm:PinHeader_1x04_P2.54mm_Vertical
- J7: footprint TerminalBlock:TerminalBlock_bornier-4_P5.08mm -> TerminalBlock_TE-Connectivity:TerminalBlock_TE_282834-4_1x04_P2.54mm_Horizontal
Connections:
- net +12P: now also J17.3 (Pin_3), R10.1, J11.7, J11.9, J6.1 (Pin_1), J8.10, J8.8; no longer J17.5 (Pin_5)
- net +12V: no longer R10.1
- net +3V3: now also J17.6 (Pin_6), JP2.1 (A), JP3.1 (A), JP5.1 (A), J11.2, J8.1, R11.2; no longer JP2.3 (B), JP3.3 (B), JP5.3 (B)
- net +5V: now also JP2.3 (B), JP3.3 (B), JP5.3 (B), J11.3, J11.5, J8.4, J8.6; no longer JP2.1 (A), JP3.1 (A), JP5.1 (A)
- net +BATT: now also TP1.1, TP3.1
- net ACCEL INT1: now also J11.17, J8.18
- net ACCEL INT2: now also J11.15, J8.16
- net ARM+: now also J6.2 (Pin_2)
- net BARO INT: now also J11.23, J8.24
- net CS SD: now also J11.13, J8.14
- net FLASH CS: now also J11.11, J8.12
- net GND: now also J17.5 (Pin_5), D3.1 (K), H13.1, H14.1, H15.1, H16.1, J11.29, J11.30, J8.29, J8.30, TP2.1
- net GYRO INT3: now also J11.19, J8.20
- net GYRO INT4: now also J11.21, J8.22
- net MISO: now also J11.24, J8.23
- net MOSI: now also J11.26, J8.25
- net P1 EN: now also J11.25, J8.26
- net P2 EN: now also J11.27, J8.28
- net PB14: now also J11.28, J8.27
- net PB15: now also J11.8, J8.7
- net PC8: now also J11.1, J8.2
- net SCK: now also J11.22, J8.21
- net SCL: now also J11.12, J8.11
- net SDA: now also J11.10, J8.9
- net SERVO1: now also J11.14, J8.13
- net SERVO2: now also J11.16, J8.15
- net SERVO3: now also J11.18, J8.17
- net SERVO4: now also J11.20, J8.19
- net TOGGLED12V: now also TP4.1
- net USART2 RX: now also J11.6, J8.5
- net USART2 TX: now also J11.4, J8.3
- new net: D3.2 (A), R11.1
- no-connect marks 15 -> 34
Other:
- moved on the sheet: C1, C2, C3, C4, R1, R3, R4, R5, R6, U1, U2
