File: avionics/hyades/hyades/hyades.kicad_sch (KiCad schematic)
At the start: 110 parts, among them J1 USB_B_Micro, J10 BOARDTOBOARDB, J11 BOARDTOBOARDF, J12 BOARDTOBOARDF, J13 BOARDTOBOARDF, J14 BOARDTOBOARDF, J15 BOARDTOBOARDB, J16 BOARDTOBOARDB, J17 Conn_02x04_Odd_Even, J18 SPI HEADER, J19 I2C HEADER, J2 Servo1, J20 UART HEADER, J3 Servo2, J4 Servo3, J5 Servo4, J6 Screw_Terminal_01x02, J7 Screw_Terminal_01x04, J8 BOARDTOBOARDB, J9 MEM2067-02-180-00-A, Q1 AO3401A, Q2 Q_NMOS_GSD, Q3 Q_NMOS_GSD, SW1 SW_MEC_5E, SW2 SW_SPDT, SW3 SW_SPDT, U1 LM317_SOT-223, U2 LM317_SOT-223, U3 USBLC6-2SC6, U4 BMI088, U5 BMP390L, U6 W25Q32JVSS, U7 STM32F405RGTx, X1 ECS-2520MV-xxx-xx

Commit message: lyra r1 work
Other:
- moved on the sheet: TP1, TP2, TP3, TP4
Changed lines of the file:
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@@
     )
   )
-  (global_label "TOGGLED12V" (shape input) (at 378.46 333.375 180) (fields_autoplaced)
+  (global_label "TOGGLED12V" (shape input) (at 350.52 339.725 180) (fields_autoplaced)
     (effects (font (size 1.27 1.27)) (justify right))
-    (property "Intersheetrefs" "${INTERSHEET_REFS}" (at 363.7614 333.375 0)
+    (property "Intersheetrefs" "${INTERSHEET_REFS}" (at 335.8214 339.725 0)
       (effects (font (size 1.27 1.27)) (justify right) hide)
     )
@@
     )
   )
-  (symbol (lib_id "Connector:TestPoint") (at 379.73 309.245 270) (unit 1)
+  (symbol (lib_id "Connector:TestPoint") (at 351.79 315.595 270) (unit 1)
     (in_bom yes) (on_board yes) (dnp no) (fields_autoplaced)
-    (property "Reference" "TP1" (at 384.81 307.975 90)
+    (property "Reference" "TP1" (at 356.87 314.325 90)
       (effects (font (size 1.27 1.27)) (justify left))
     )
-    (property "Value" "Connector" (at 384.81 310.515 90)
+    (property "Value" "Connector" (at 356.87 316.865 90)
       (effects (font (size 1.27 1.27)) (justify left))
     )
-    (property "Footprint" "TestPoint:TestPoint_Keystone_5019_Minature" (at 379.73 314.325 0)
+    (property "Footprint" "TestPoint:TestPoint_Keystone_5019_Minature" (at 351.79 320.675 0)
       (effects (font (size 1.27 1.27)) hide)
     )
-    (property "Datasheet" "~" (at 379.73 314.325 0)
+    (property "Datasheet" "~" (at 351.79 320.675 0)
       (effects (font (size 1.27 1.27)) hide)
     )
@@
     )
   )
-  (symbol (lib_id "Connector:TestPoint") (at 379.73 313.055 270) (unit 1)
+  (symbol (lib_id "Connector:TestPoint") (at 351.79 319.405 270) (unit 1)
     (in_bom yes) (on_board yes) (dnp no) (fields_autoplaced)
-    (property "Reference" "TP2" (at 384.81 311.785 90)
+    (property "Reference" "TP2" (at 356.87 318.135 90)
       (effects (font (size 1.27 1.27)) (justify left))
     )
-    (property "Value" "Connector" (at 384.81 314.325 90)
+    (property "Value" "Connector" (at 356.87 320.675 90)
       (effects (font (size 1.27 1.27)) (justify left))
     )
-    (property "Footprint" "TestPoint:TestPoint_Keystone_5019_Minature" (at 379.73 318.135 0)
+    (property "Footprint" "TestPoint:TestPoint_Keystone_5019_Minature" (at 351.79 324.485 0)
       (effects (font (size 1.27 1.27)) hide)
     )
-    (property "Datasheet" "~" (at 379.73 318.135 0)
+    (property "Datasheet" "~" (at 351.79 324.485 0)
       (effects (font (size 1.27 1.27)) hide)
     )
@@
     )
   )
-  (symbol (lib_id "power:+BATT") (at 378.46 329.565 90) (unit 1)
+  (symbol (lib_id "power:+BATT") (at 350.52 335.915 90) (unit 1)
     (in_bom yes) (on_board yes) (dnp no) (fields_autoplaced)
-    (property "Reference" "#PWR01" (at 382.27 329.565 0)
+    (property "Reference" "#PWR01" (at 354.33 335.915 0)
       (effects (font (size 1.27 1.27)) hide)
     )
-    (property "Value" "+BATT" (at 374.65 330.2 90)
+    (property "Value" "+BATT" (at 346.71 336.55 90)
       (effects (font (size 1.27 1.27)) (justify left))
     )
-    (property "Footprint" "" (at 378.46 329.565 0)
+    (property "Footprint" "" (at 350.52 335.915 0)
       (effects (font (size 1.27 1.27)) hide)
     )
-    (property "Datasheet" "" (at 378.46 329.565 0)
+    (property "Datasheet" "" (at 350.52 335.915 0)
       (effects (font (size 1.27 1.27)) hide)
     )
@@
     )
   )
-  (symbol (lib_id "Connector:TestPoint") (at 378.46 333.375 270) (unit 1)
+  (symbol (lib_id "Connector:TestPoint") (at 350.52 339.725 270) (unit 1)
     (in_bom yes) (on_board yes) (dnp no) (fields_autoplaced)
-    (property "Reference" "TP4" (at 383.54 332.105 90)
+    (property "Reference" "TP4" (at 355.6 338.455 90)
       (effects (font (size 1.27 1.27)) (justify left))
     )
-    (property "Value" "Connector" (at 383.54 334.645 90)
+    (property "Value" "Connector" (at 355.6 340.995 90)
       (effects (font (size 1.27 1.27)) (justify left))
     )
-    (property "Footprint" "TestPoint:TestPoint_Keystone_5019_Minature" (at 378.46 338.455 0)
+    (property "Footprint" "TestPoint:TestPoint_Keystone_5019_Minature" (at 350.52 344.805 0)
       (effects (font (size 1.27 1.27)) hide)
     )
-    (property "Datasheet" "~" (at 378.46 338.455 0)
+    (property "Datasheet" "~" (at 350.52 344.805 0)
       (effects (font (size 1.27 1.27)) hide)
     )
@@
     )
   )
-  (symbol (lib_id "power:GND") (at 379.73 313.055 270) (unit 1)
+  (symbol (lib_id "power:GND") (at 351.79 319.405 270) (unit 1)
     (in_bom yes) (on_board yes) (dnp no) (fields_autoplaced)
-    (property "Reference" "#PWR039" (at 373.38 313.055 0)
+    (property "Reference" "#PWR039" (at 345.44 319.405 0)
       (effects (font (size 1.27 1.27)) hide)
     )
-    (property "Value" "GND" (at 375.92 313.055 90)
+    (property "Value" "GND" (at 347.98 319.405 90)
       (effects (font (size 1.27 1.27)) (justify right))
     )
-    (property "Footprint" "" (at 379.73 313.055 0)
+    (property "Footprint" "" (at 351.79 319.405 0)
       (effects (font (size 1.27 1.27)) hide)
     )
-    (property "Datasheet" "" (at 379.73 313.055 0)
+    (property "Datasheet" "" (at 351.79 319.405 0)
       (effects (font (size 1.27 1.27)) hide)
     )
@@
     )
   )
-  (symbol (lib_id "power:+BATT") (at 379.73 309.245 90) (unit 1)
+  (symbol (lib_id "power:+BATT") (at 351.79 315.595 90) (unit 1)
     (in_bom yes) (on_board yes) (dnp no) (fields_autoplaced)
-    (property "Reference" "#PWR01" (at 383.54 309.245 0)
+    (property "Reference" "#PWR01" (at 355.6 315.595 0)
       (effects (font (size 1.27 1.27)) hide)
     )
-    (property "Value" "+BATT" (at 375.92 309.88 90)
+    (property "Value" "+BATT" (at 347.98 316.23 90)
       (effects (font (size 1.27 1.27)) (justify left))
     )
-    (property "Footprint" "" (at 379.73 309.245 0)
+    (property "Footprint" "" (at 351.79 315.595 0)
       (effects (font (size 1.27 1.27)) hide)
     )
-    (property "Datasheet" "" (at 379.73 309.245 0)
+    (property "Datasheet" "" (at 351.79 315.595 0)
       (effects (font (size 1.27 1.27)) hide)
     )
@@
     )
   )
-  (symbol (lib_id "Connector:TestPoint") (at 378.46 329.565 270) (unit 1)
+  (symbol (lib_id "Connector:TestPoint") (at 350.52 335.915 270) (unit 1)
     (in_bom yes) (on_board yes) (dnp no) (fields_autoplaced)
-    (property "Reference" "TP3" (at 383.54 328.295 90)
+    (property "Reference" "TP3" (at 355.6 334.645 90)
       (effects (font (size 1.27 1.27)) (justify left))
     )
-    (property "Value" "Connector" (at 383.54 330.835 90)
+    (property "Value" "Connector" (at 355.6 337.185 90)
       (effects (font (size 1.27 1.27)) (justify left))
     )
-    (property "Footprint" "TestPoint:TestPoint_Keystone_5019_Minature" (at 378.46 334.645 0)
+    (property "Footprint" "TestPoint:TestPoint_Keystone_5019_Minature" (at 350.52 340.995 0)
       (effects (font (size 1.27 1.27)) hide)
     )
-    (property "Datasheet" "~" (at 378.46 334.645 0)
+    (property "Datasheet" "~" (at 350.52 340.995 0)
       (effects (font (size 1.27 1.27)) hide)
     )
