File: avionics/kicad/Lyra_flight_computer/Lyra v2/Lyra V2/Lyra V2.kicad_pcb (KiCad board)
At the start: 4 copper layers, 40 x 75 mm, 90 parts, among them J1 USB_B_Micro, J10 Conn_01x04, J11 Conn_01x04, J12 Conn_01x03, J13 MEM2067-02-180-00-A, J2 Screw_Terminal_01x04, J3 Screw_Terminal_01x04, J4 Conn_02x03_Odd_Even, J5 Screw_Terminal_01x04, J6 Screw_Terminal_01x04, J7 Conn_02x03_Odd_Even, J8 Conn_02x03_Odd_Even, J9 Conn_02x03_Odd_Even, Q1 AO3401A, Q2 BSS138, Q3 BSS138, SW1 SW_Push_DPDT, U1 AZ1117-3.3, U2 AZ1117-5.0, U3 LIS3MDL, U4 BMP390L, U5 W25Q128JVS, U6 RP2040, U7 BMI088, X1 ECS-2520MV-xxx-xx

Commit message: lots of things
Parts:
- moved R12 15.9 mm to (123.8, 105.3), turned to 180 degrees
- moved D3 12.5 mm to (123.7, 103.1), turned to 180 degrees
- moved C27 9.97 mm to (115.7, 95.7), turned to 180 degrees
- moved C23 9.57 mm to (125.6, 96.4), turned to 0 degrees
- moved R16 8.72 mm to (112.8, 94.1), turned to 180 degrees
- moved R15 8.65 mm to (112.8, 95.7), turned to 0 degrees
- moved C30 8.15 mm to (117.3, 98.7), turned to 90 degrees
- moved C21 7.55 mm to (114.4, 94.2), turned to 180 degrees
- moved C20 6.94 mm to (117.6, 94.2), turned to 0 degrees
- moved R14 6.84 mm to (116.9, 101.6), turned to 180 degrees
- moved C15 5.70 mm to (118.7, 96.5), turned to 0 degrees
- moved C17 5.67 mm to (122.6, 95.7), turned to 180 degrees
- moved C18 5.63 mm to (111.3, 90.5)
- moved U5 5.52 mm to (110.1, 95.9)
- moved D2 4.81 mm to (110.4, 105.6)
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Connections:
- net Net-(U6-USB_DM) renamed /RP USB_D-
- net Net-(U6-USB_DP) renamed /RP USB_D+
- J10 pad 2: /I2C1 SDA -> /I2C1 SCL
- J10 pad 3: /I2C1 SCL -> /I2C1 SDA
Routing:
- net +5V: track 147.5 -> 190.5 mm, vias 9 -> 5
- net /P1 CONT: track 60.4 -> 87.8 mm, vias 1 -> 3
- net /QSPI_SS: track 40.9 -> 21.9 mm, vias 5 -> 2
- net /SPI0 MISO: track 58.0 -> 42.3 mm, vias 2 -> 1
- net /SPI0 MOSI: track 48.1 -> 32.6 mm
- net /MAG DRDY: track 57.4 -> 42.1 mm, vias 8 -> 2
- net /SPI0 SCLK: track 59.6 -> 44.6 mm, vias 1 -> 2
- net /P2 CONT: track 72.1 -> 85.8 mm, vias 1 -> 3
- net GND: track 70.6 -> 58.9 mm, vias 44 -> 41
- net /USB_D-: track 17.9 -> 6.73 mm
- net /USB_D+: track 17.6 -> 6.77 mm
- net /BRKOUT CS: track 36.6 -> 25.8 mm, vias 1 -> 2
- net /I2C1 SDA: track 52.8 -> 43.0 mm, vias 2 -> 4
- net +12P: track 92.4 -> 101.9 mm
- net /PYRO PWR: track 64.5 -> 72.9 mm, vias 3 -> 1
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
Commit message: buncho stuf
Parts:
- moved J2 15.3 mm to (103.8, 71.4), turned to -90 degrees
- moved R15 0.96 mm to (113.7, 95.6)
- moved R16 0.96 mm to (113.7, 94.1)
- moved J5 0.22 mm to (136.0, 86.5)
- moved J4 0.20 mm to (135.4, 103.1)
- moved J6 0.18 mm to (136.0, 112.8)
- moved J3 0.13 mm to (103.9, 112.7)
- moved J11 0.13 mm to (129.1, 98.9)
- moved C9 0.10 mm to (132.8, 101.9)
- moved J10 0.10 mm to (109.8, 71.8)
- moved R12 0.08 mm to (123.7, 105.3)
- moved D3 0.08 mm to (123.7, 103.1)
- moved J8 0.07 mm to (133.0, 93.8)
Connections:
- J2 pad 2: +12P -> +3V3
- J2 pad 3: +5V -> GND
- J2 pad 4: GND -> +12P
- J5 pad 1: +3V3 -> /PYRO PWR
- J5 pad 2: GND -> +12P
- J5 pad 3: /PYRO PWR -> GND
- J5 pad 4: +12P -> +5V
Routing:
- net +12VA: track 38.2 -> 19.5 mm
- net /PYRO PWR: track 72.9 -> 58.2 mm
- net +3V3: track 60.9 -> 48.6 mm
- net /GPIO26: track 18.9 -> 29.7 mm
- net +5V: track 190.5 -> 182.2 mm
- net +12P: track 101.9 -> 109.8 mm
- net +BATT: track 33.0 -> 37.8 mm
- net /USB_D-: track 6.73 -> 7.84 mm
- net /USB_D+: track 6.77 -> 7.87 mm
- net /RP USB_D+: track 3.12 -> 2.07 mm
- net /RP USB_D-: track 3.14 -> 2.11 mm
- added copper zone on B.Cu, net +12VA
- added copper zone on F.Cu, net +3V3
- added copper zone on F.Cu, net +5V
Other:
- board text added: "5V GND ARM+ ARM-"
- board text added: "D26 3V3 GND 12V"
- board text added: "JLCJLCJLCJLC"
- board text removed: "ARM+ ARM- GND 3V3"
- board text removed: "GND 5V 12P D26"
