File: avionics/kicad/Lyra_flight_computer/Lyra v2/Lyra V2/Lyra V2.kicad_sch (KiCad schematic)
At the start: 90 parts, among them J1 USB_B_Micro, J10 Conn_01x04, J11 Conn_01x04, J12 Conn_01x03, J2 Screw_Terminal_01x04, J3 Screw_Terminal_01x04, J4 Conn_02x03_Odd_Even, J5 Screw_Terminal_01x04, J6 Screw_Terminal_01x04, J7 Conn_02x03_Odd_Even, J8 Conn_02x03_Odd_Even, J9 Conn_02x03_Odd_Even, J9 MEM2067-02-180-00-A, Q1 AO3401A, Q2 BSS138, Q3 BSS138, SW1 SW_Push_DPDT, U1 AZ1117-3.3, U2 AZ1117-5.0, U3 LIS3MDL, U4 BMP390L, U5 W25Q128JVS, U6 RP2040, U7 BMI088, X1 ECS-2520MV-xxx-xx

Commit message: lots of things
Connections:
- net I2C1 SCL: now also J10.2 (Pin_2); no longer J10.3 (Pin_3)
- net I2C1 SDA: now also J10.3 (Pin_3); no longer J10.2 (Pin_2)
- net RP USB_D+: now reaches R15.2, U6.47 (USB_DP)
- net RP USB_D-: now reaches R16.1, U6.46 (USB_DM)
Other:
- moved on the sheet: R15, R16
Changed lines of the file:
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@@
     (stroke (width 0) (type default))
   )
-  (wire (pts (xy 312.42 167.005) (xy 323.215 167.005))
+  (wire (pts (xy 302.26 167.005) (xy 313.055 167.005))
     (stroke (width 0) (type default))
   )
@@
     (stroke (width 0) (type default))
   )
-  (wire (pts (xy 312.42 164.465) (xy 323.215 164.465))
+  (wire (pts (xy 302.26 164.465) (xy 313.055 164.465))
     (stroke (width 0) (type default))
   )
@@
     (stroke (width 0) (type default))
   )
+  (wire (pts (xy 318.135 164.465) (xy 331.47 164.465))
+    (stroke (width 0) (type default))
+  )
   (wire (pts (xy 307.34 62.865) (xy 308.61 62.865))
     (stroke (width 0) (type default))
@@
     (stroke (width 0) (type default))
   )
-  (wire (pts (xy 328.295 164.465) (xy 331.47 164.465))
-    (stroke (width 0) (type default))
-  )
   (wire (pts (xy 308.61 57.785) (xy 307.34 57.785))
     (stroke (width 0) (type default))
@@
     (stroke (width 0) (type default))
   )
-  (wire (pts (xy 328.295 167.005) (xy 331.47 167.005))
+  (wire (pts (xy 318.135 167.005) (xy 331.47 167.005))
     (stroke (width 0) (type default))
   )
@@
     (effects (font (size 1.27 1.27)) (justify right bottom))
   )
+  (label "RP USB_D-" (at 321.945 167.005 0) (fields_autoplaced)
+    (effects (font (size 1.27 1.27)) (justify left bottom))
+  )
   (label "RUN" (at 278.765 172.72 0) (fields_autoplaced)
     (effects (font (size 1.27 1.27)) (justify left bottom))
   )
-  (label "I2C1 SCL" (at 179.705 180.34 0) (fields_autoplaced)
+  (label "I2C1 SCL" (at 179.705 177.8 0) (fields_autoplaced)
     (effects (font (size 1.27 1.27)) (justify left bottom))
   )
@@
     (effects (font (size 1.27 1.27)) (justify left bottom))
   )
-  (label "USB_D+" (at 312.42 164.465 0) (fields_autoplaced)
+  (label "USB_D+" (at 302.26 164.465 0) (fields_autoplaced)
     (effects (font (size 1.27 1.27)) (justify left bottom))
   )
@@
     (effects (font (size 1.27 1.27)) (justify left bottom))
   )
+  (label "RP USB_D+" (at 321.945 164.465 0) (fields_autoplaced)
+    (effects (font (size 1.27 1.27)) (justify left bottom))
+  )
   (label "PYRO PWR" (at 99.06 263.525 0) (fields_autoplaced)
     (effects (font (size 1.27 1.27)) (justify left bottom))
@@
     (effects (font (size 1.27 1.27)) (justify right bottom))
   )
-  (label "USB_D-" (at 312.42 167.005 0) (fields_autoplaced)
+  (label "USB_D-" (at 302.26 167.005 0) (fields_autoplaced)
     (effects (font (size 1.27 1.27)) (justify left bottom))
   )
@@
     (effects (font (size 1.27 1.27)) (justify right bottom))
   )
-  (label "I2C1 SDA" (at 179.705 177.8 0) (fields_autoplaced)
+  (label "I2C1 SDA" (at 179.705 180.34 0) (fields_autoplaced)
     (effects (font (size 1.27 1.27)) (justify left bottom))
   )
@@
     )
   )
-  (symbol (lib_id "Device:R_Small") (at 325.755 164.465 90) (unit 1)
+  (symbol (lib_id "Device:R_Small") (at 315.595 164.465 90) (unit 1)
     (in_bom yes) (on_board yes) (dnp no) (fields_autoplaced)
-    (property "Reference" "R15" (at 325.755 159.385 90)
+    (property "Reference" "R15" (at 315.595 159.385 90)
       (effects (font (size 1.27 1.27)))
     )
-    (property "Value" "27R" (at 325.755 161.925 90)
+    (property "Value" "27R" (at 315.595 161.925 90)
       (effects (font (size 1.27 1.27)))
     )
-    (property "Footprint" "Resistor_SMD:R_0603_1608Metric" (at 325.755 164.465 0)
+    (property "Footprint" "Resistor_SMD:R_0603_1608Metric" (at 315.595 164.465 0)
       (effects (font (size 1.27 1.27)) hide)
     )
-    (property "Datasheet" "~" (at 325.755 164.465 0)
+    (property "Datasheet" "~" (at 315.595 164.465 0)
       (effects (font (size 1.27 1.27)) hide)
     )
@@
     )
   )
-  (symbol (lib_id "Device:R_Small") (at 325.755 167.005 270) (unit 1)
+  (symbol (lib_id "Device:R_Small") (at 315.595 167.005 270) (unit 1)
     (in_bom yes) (on_board yes) (dnp no)
-    (property "Reference" "R16" (at 325.755 171.45 90)
+    (property "Reference" "R16" (at 315.595 171.45 90)
       (effects (font (size 1.27 1.27)))
     )
-    (property "Value" "27R" (at 325.755 169.545 90)
+    (property "Value" "27R" (at 315.595 169.545 90)
       (effects (font (size 1.27 1.27)))
     )
-    (property "Footprint" "Resistor_SMD:R_0603_1608Metric" (at 325.755 167.005 0)
+    (property "Footprint" "Resistor_SMD:R_0603_1608Metric" (at 315.595 167.005 0)
       (effects (font (size 1.27 1.27)) hide)
     )
-    (property "Datasheet" "~" (at 325.755 167.005 0)
+    (property "Datasheet" "~" (at 315.595 167.005 0)
       (effects (font (size 1.27 1.27)) hide)
     )

Commit message: buncho stuf
Parts:
- C26, C28: value 100nf -> 100n
- R12: value R_Small -> 1k
Connections:
- net +12P: now also J2.4 (Pin_4), J5.2 (Pin_2); no longer J2.2 (Pin_2), J5.4 (Pin_4)
- net +3V3: now also J2.2 (Pin_2); no longer J5.1 (Pin_1)
- net +5V: now also J5.4 (Pin_4); no longer J2.3 (Pin_3)
- net GND: now also J2.3 (Pin_3), J5.3 (Pin_3); no longer J2.4 (Pin_4), J5.2 (Pin_2)
- net PYRO PWR: now also J5.1 (Pin_1); no longer J5.3 (Pin_3)
