File: Sierra Coyote/P&ID/pid/pid.kicad_sch (KiCad schematic)
At the start: 9 parts

Commit message: hm
Parts:
- renumbered GasBottle1 to N2O, Tank_Slim_4Port1 to Tank1, igniter1 to ignitercartridge
Connections:
- net at Hose1.~: now also SV1.; no longer CheckValve1.~
- net at SV1.: now also N2O.~; no longer Hose1.~
- net at Tank1.~: now also SV2.; no longer SV3.
- net at SV2.: now also Engine1.~ (O); no longer Tank1.~
- new net: CheckValve1.~, Hose1.~
- new net: SV3., Tank1.~
Changed lines of the file:
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@@
 			(width 0)
 			(type default)
+			(color 0 194 0 1)
 		)
 	)
@@
 			(width 0)
 			(type default)
+			(color 194 0 0 1)
 		)
 	)
@@
 			(width 0)
 			(type default)
+			(color 0 194 0 1)
 		)
 	)
@@
 			(width 0)
 			(type default)
+			(color 194 0 0 1)
 		)
 	)
@@
 			(width 0)
 			(type default)
+			(color 0 194 0 1)
 		)
 	)
@@
 			(width 0)
 			(type default)
+			(color 0 194 0 1)
 		)
 	)
@@
 			(width 0)
 			(type default)
+			(color 0 194 0 1)
 		)
 	)
@@
 			(width 0)
 			(type default)
+			(color 194 0 0 1)
 		)
 	)
@@
 			(width 0)
 			(type default)
+			(color 0 194 0 1)
 		)
 	)
@@
 			(width 0)
 			(type default)
+			(color 194 0 0 1)
 		)
 	)
@@
 			(width 0)
 			(type default)
+			(color 194 0 0 1)
 		)
 	)
@@
 			(width 0)
 			(type default)
+			(color 0 194 0 1)
 		)
 	)
@@
 			(width 0)
 			(type default)
+			(color 0 194 0 1)
 		)
 	)
@@
 			(width 0)
 			(type default)
+			(color 194 0 0 1)
 		)
 	)
@@
 			(width 0)
 			(type default)
+			(color 0 194 0 1)
 		)
 	)
@@
 			(width 0)
 			(type default)
+			(color 194 0 0 1)
 		)
 	)
@@
 			(width 0)
 			(type default)
+			(color 0 194 0 1)
 		)
 	)
@@
 			(width 0)
 			(type default)
+			(color 194 0 0 1)
 		)
 	)
@@
 			(width 0)
 			(type default)
+			(color 0 194 0 1)
+		)
+	)
+	(netclass_flag ""
+		(length 2.54)
+		(shape round)
+		(at 100.33 85.09 0)
+		(fields_autoplaced yes)
+		(effects
+			(font
+				(size 1.27 1.27)
+			)
+			(justify left bottom)
+		)
+		(property "Netclass" "OX"
+			(at 101.0285 82.55 0)
+			(effects
+				(font
+					(size 1.27 1.27)
+					(italic yes)
+				)
+				(justify left)
+			)
 		)
 	)
@@
 		(on_board yes)
 		(dnp no)
-		(fields_autoplaced yes)
-		(property "Reference" "igniter1"
-			(at 131.826 100.33 0)
-			(effects
-				(font
-					(size 0.508 0.508)
-				)
-				(hide yes)
+		(property "Reference" "ignitercartridge"
+			(at 113.538 105.156 90)
+			(effects
+				(font
+					(size 1 1)
+				)
+				(justify left)
 			)
 		)
@@
 			(project "pid"
 				(path "/dc29bb4e-9c9a-4427-b7c6-9d7a2377948e"
-					(reference "igniter1")
+					(reference "ignitercartridge")
 					(unit 1)
 				)
@@
 		(on_board yes)
 		(dnp no)
-		(fields_autoplaced yes)
-		(property "Reference" "Tank_Slim_4Port1"
-			(at 143.51 66.675 0)
-			(effects
-				(font
-					(size 0.508 0.508)
+		(property "Reference" "Tank1"
+			(at 124.46 67.31 0)
+			(effects
+				(font
+					(size 1 1)
 				)
 				(justify left)
@@
 				)
 				(justify left)
+				(hide yes)
 			)
 		)
@@
 			(project "pid"
 				(path "/dc29bb4e-9c9a-4427-b7c6-9d7a2377948e"
-					(reference "Tank_Slim_4Port1")
+					(reference "Tank1")
 					(unit 1)
 				)
@@
 		(on_board yes)
 		(dnp no)
-		(fields_autoplaced yes)
-		(property "Reference" "GasBottle1"
-			(at 91.44 101.6 0)
-			(effects
-				(font
-					(size 0.508 0.508)
+		(property "Reference" "N2O"
+			(at 83.566 101.854 0)
+			(effects
+				(font
+					(size 1 1)
 				)
 				(justify left)
@@
 			(project "pid"
 				(path "/dc29bb4e-9c9a-4427-b7c6-9d7a2377948e"
-					(reference "GasBottle1")
+					(reference "N2O")
 					(unit 1)
 				)
@@
 		(on_board yes)
 		(dnp no)
-		(fields_autoplaced yes)
 		(property "Reference" "SV3"
-			(at 135.128 99.06 0)
-			(effects
-				(font
-					(size 0.508 0.508)
-				)
+			(at 133.858 99.06 90)
+			(effects
+				(font
+					(size 1 1)
+				)
+				(justify left)
 			)
 		)
@@
 		(fields_autoplaced yes)
 		(property "Reference" "SV1"
-			(at 92.71 88.392 0)
-			(effects
-				(font
-					(size 0.508 0.508)
+			(at 92.71 77.47 0)
+			(effects
+				(font
+					(size 1 1)
 				)
 			)
@@
 		(fields_autoplaced yes)
 		(property "Reference" "SV2"
-			(at 143.51 54.102 0)
-			(effects
-				(font
-					(size 0.508 0.508)
-				)
-			)
+			(at 143.51 43.18 0)
+			(effects
+				(font
+					(size 1 1)
+				)
+			)
