File: CAD/JUMP/wiring/sustainer harness diagram/JUMP sustainer wiring/JUMP sustainer wiring.kicad_sch (KiCad schematic)
At the start: 26 parts, among them SW1 SW_SPDT, SW2 SW_SPDT, SW3 SW_SPDT, SW5 SW_SPST, SW6 SW_SPDT

Commit message: phone holder, payload cad, etc
Connections:
- net at TM1.5 (BATT-): now also BT7.2 (-); no longer MAG2.6 (OUT+)
- net at TM1.6 (BATT+): now also BT7.1 (+)
- net at MAG2.5 (OUT-): no longer TM1.6 (BATT+)
- new net: MAG2.6 (OUT+), TM1.5 (BATT-)
- new net: MAG2.5 (OUT-), TM1.6 (BATT+)
- no-connect marks 6 -> 7
Other:
- note added: "2P PH"
- moved on the sheet: BT2, BT3, BT6, EMATCH4, FWGPS1, RTD1, SPLIT1
