File: CAD/Leap of faith/sustainer/avionics/Bulkhead PCB/bulkhead pcb/bulkhead pcb.kicad_pcb (KiCad board)
At the start: 2 copper layers, 48 x 48 mm, 18 parts, among them J1 Conn_01x04, J10 Conn_01x02, J11 Conn_01x02, J12 Conn_01x02, J2 Conn_01x02, J3 Conn_01x02, J8 Conn_01x02, J9 Conn_01x02, SW1 SW_SPDT, SW3 SW_SPDT, U1 RS6651

Commit message: backplane and johnnie
Parts:
- removed J10, J11, J12, J9: Conn_01x02, Connector_PinSocket_2.54mm:PinSocket_1x02_P2.54mm_Vertical
- removed J3, J8: Conn_01x02, Connector_JST:JST_PH_B2B-PH-K_1x02_P2.00mm_Vertical
- added C4: 100n, Capacitor_SMD:C_0603_1608Metric, B.Cu at (114.6, 97.4)
- added J4: Conn_02x04_Odd_Even, Connector_PinHeader_2.54mm:PinHeader_2x04_P2.54mm_Vertical, B.Cu at (112.0, 115.6)
- added J5: Conn_01x02, Connector_JST:JST_PH_B2B-PH-K_1x02_P2.00mm_Vertical, F.Cu at (97.0, 83.8)
- added J6: Conn_01x02, Connector_JST:JST_PH_B2B-PH-K_1x02_P2.00mm_Vertical, F.Cu at (104.4, 83.8)
- added JP1: SolderJumper_2_Open, Jumper:SolderJumper-2_P1.3mm_Open_Pad1.0x1.5mm, F.Cu at (98.2, 109.6)
- added JP2: SolderJumper_2_Open, Jumper:SolderJumper-2_P1.3mm_Open_Pad1.0x1.5mm, F.Cu at (98.2, 107.6)
- added JP3: SolderJumper_3_Open, Jumper:SolderJumper-3_P1.3mm_Open_RoundedPad1.0x1.5mm, F.Cu at (103.6, 101.3)
- L1: footprint Inductor_SMD:L_1210_3225Metric -> Inductor_SMD:L_Chilisin_BWVS00505020
- R1: value 0 -> 1k
- SW1, SW3: footprint Button_Switch_THT:SW_XKB_DM1-16UC-1 -> pullpinswitches:OMRON D2F-F-A1; moved to B.Cu
- moved SW3 63.0 mm to (108.8, 98.3)
- moved SW1 52.6 mm to (93.3, 104.8), turned to 0 degrees
- moved R1 46.7 mm to (111.6, 97.4)
- moved J1 44.8 mm to (94.3, 117.1), turned to 0 degrees
- moved C2 43.8 mm to (114.6, 100.4)
- moved C1 43.7 mm to (113.0, 97.4)
- moved C3 43.7 mm to (113.0, 100.4)
- moved R2 43.7 mm to (115.5, 102.7)
- moved R3 43.7 mm to (118.5, 102.7)
- moved U1 43.7 mm to (117.7, 99.6)
- moved L1 43.7 mm to (118.2, 94.9)
- moved J2 28.9 mm to (107.3, 118.3), turned to 180 degrees
Connections:
- SW1 pad 1: /Raven Arm+ -> Net-(JP1-B)
- SW1 pad 3: /Raven Ignitor -> Net-(JP2-B)
- SW3 pad 1: /CAM BATT POST SW -> Net-(JP3-B)
- SW3 pad 3: unconnected-(SW3-C-Pad3) -> Net-(JP3-A)
Routing:
- net /Raven Ignitor: track 0.00 -> 46.8 mm, vias 0 -> 1
- net /Raven Drogue: track 0.02 -> 28.8 mm
- net /Raven Arm+: track 0.00 -> 22.0 mm
- net /Raven Main: track 0.00 -> 20.5 mm
- net /Sustainer Ignitor: track 0.00 -> 18.7 mm
- net /CAM OUT +: track 14.0 -> 31.9 mm
- net /CAM BATT +: track 4.43 -> 17.3 mm
- net /Bulk Raven Arm+: track 0.00 -> 11.5 mm
- net /CAM BATT -: track 33.1 -> 43.5 mm
- net Net-(JP1-B): track 0.00 -> 7.09 mm
- net /CAM BATT POST SW: track 28.5 -> 22.2 mm, vias 3 -> 2
- net /Bulk Raven Drogue: track 0.00 -> 5.84 mm
- net Net-(JP3-B): track 0.00 -> 5.23 mm
- net Net-(JP2-B): track 0.00 -> 5.09 mm
- net Net-(JP3-A): track 0.00 -> 4.98 mm
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- removed copper zone on F.Cu, net /CAM BATT -
Other:
- board size 48 x 48 mm -> 44.4 x 44.4 mm

Commit message: thing
Parts:
- R1: value 1k -> 0
- moved R1 10.8 mm to (122.0, 100.0), turned to -90 degrees
- moved JP2 2.29 mm to (100.5, 107.4)
- moved JP1 2.29 mm to (100.4, 110.0)
- moved SW1 2.07 mm to (95.4, 104.6)
- moved C3 1.72 mm to (114.7, 101.0)
- moved C1 1.68 mm to (114.7, 97.8)
- moved C2 1.54 mm to (113.2, 101.0)
- moved C4 1.49 mm to (113.2, 97.8)
- moved R3 1.00 mm to (119.4, 103.3)
- moved R2 0.90 mm to (116.2, 103.3)
- moved U1 0.86 mm to (118.4, 100.1)
- moved L1 0.72 mm to (118.5, 95.5)
- moved JP3 0.28 mm to (103.5, 101.1)
Connections:
- J5 pad 1: /CAM BATT + -> /CAM BATT -
- J5 pad 2: /CAM BATT - -> /CAM BATT +
- J6 pad 1: /CAM OUT + -> /CAM BATT -
- J6 pad 2: /CAM BATT - -> /CAM OUT +
Routing:
- net /CAM BATT POST SW: track 22.2 -> 44.5 mm
- net Net-(U1-EN): track 21.5 -> 2.63 mm
- net /CAM BATT -: track 43.5 -> 31.1 mm, vias 4 -> 22
- net Net-(JP1-B): track 7.09 -> 9.45 mm
- net /Sustainer Ignitor: track 18.7 -> 16.7 mm
- net /CAM BATT +: track 17.3 -> 18.6 mm
- net /Raven Arm+: track 22.0 -> 20.7 mm
- net /CAM OUT +: track 31.9 -> 30.6 mm
- net /Raven Ignitor: track 46.8 -> 46.3 mm
- net Net-(JP2-B): track 5.09 -> 5.60 mm
- added copper zone on B.Cu, net /CAM BATT -
- added copper zone on F.Cu, net /CAM BATT -
Other:
- board text added: "JLCJLCJLCJLC"
- board text added: "YOU MIGHT THINK, WHAT IF I FALL? WELL, WHAT IF YOU DONT? WHAT IF YOU FLY?"
