File: CAD/Leap of faith/sustainer/avionics/Bulkhead PCB/bulkhead pcb/bulkhead pcb.kicad_sch (KiCad schematic)
At the start: 18 parts, among them J1 Conn_01x04, J10 Conn_01x02, J11 Conn_01x02, J12 Conn_01x02, J2 Conn_01x02, J3 Conn_01x02, J8 Conn_01x02, J9 Conn_01x02, SW1 SW_SPDT, SW3 SW_SPDT, U1 RS6651

Commit message: backplane and johnnie
Parts:
- removed J10, J11, J12, J9: Conn_01x02, Connector_PinSocket_2.54mm:PinSocket_1x02_P2.54mm_Vertical, symbol Connector_Generic:Conn_01x02
- removed J3, J8: Conn_01x02, Connector_JST:JST_PH_B2B-PH-K_1x02_P2.00mm_Vertical, symbol Connector_Generic:Conn_01x02
- added C4: 100n, Capacitor_SMD:C_0603_1608Metric, symbol Device:C_Small
- added J4: Conn_02x04_Odd_Even, Connector_PinHeader_2.54mm:PinHeader_2x04_P2.54mm_Vertical, symbol Connector_Generic:Conn_02x04_Odd_Even
- added J5, J6: Conn_01x02, Connector_JST:JST_PH_B2B-PH-K_1x02_P2.00mm_Vertical, symbol Connector_Generic:Conn_01x02
- added JP1, JP2: SolderJumper_2_Open, Jumper:SolderJumper-2_P1.3mm_Open_Pad1.0x1.5mm, symbol Jumper:SolderJumper_2_Open
- added JP3: SolderJumper_3_Open, Jumper:SolderJumper-3_P1.3mm_Open_RoundedPad1.0x1.5mm, symbol Jumper:SolderJumper_3_Open
- L1: footprint Inductor_SMD:L_1210_3225Metric -> Inductor_SMD:L_Chilisin_BWVS00505020
- R1: value 0 -> 1k
- SW1, SW3: footprint Button_Switch_THT:SW_XKB_DM1-16UC-1 -> pullpinswitches:OMRON D2F-F-A1
Connections:
- net Bulk Raven Arm+: now also J4.2 (Pin_2)
- net Bulk Raven Drogue: now also J4.1 (Pin_1)
- net CAM BATT +: now also J5.1 (Pin_1)
- net CAM BATT -: now also C4.2, J5.2 (Pin_2), J6.2 (Pin_2)
- net CAM BATT POST SW: now also C4.1, JP3.2 (C); no longer SW3.1 (A)
- net CAM OUT +: now also J6.1 (Pin_1)
- net Raven Arm+: now also J4.3 (Pin_3), J4.4 (Pin_4), JP1.1 (A); no longer SW1.1 (A)
- net Raven Drogue: now also J4.6 (Pin_6)
- net Raven Ignitor: now also J4.7 (Pin_7), JP2.1 (A); no longer SW1.3 (C)
- net Raven Main: now also J4.5 (Pin_5)
- net Sustainer Ignitor: now also J4.8 (Pin_8)
- net at SW3.3 (C): now also JP3.1 (A)
- new net: JP2.2 (B), SW1.3 (C)
- new net: JP3.3 (B), SW3.1 (A)
- new net: JP1.2 (B), SW1.1 (A)
- no-connect marks 1 -> 0
Other:
- moved on the sheet: C1

Commit message: thing
Parts:
- R1: value 1k -> 0
Connections:
- net CAM BATT +: now also J5.2 (Pin_2); no longer J5.1 (Pin_1)
- net CAM BATT -: now also J5.1 (Pin_1), J6.1 (Pin_1); no longer J5.2 (Pin_2), J6.2 (Pin_2)
- net CAM OUT +: now also J6.2 (Pin_2); no longer J6.1 (Pin_1)
